Commit message: Added camera ray at the robot front; reduced max range of lidars to 5m (temporarily); prepped for outdoor cases

File: description/camera_ray.xacro (robot description, xacro)
@@ -1,15 +1,15 @@
 <?xml version="1.0"?>
 <robot xmlns:xacro="http://www.ros.org/wiki/xacro" >
-    <joint name="lidar_l_joint" type="fixed">
+    <joint name="camera_ray_joint" type="fixed">
         <parent link="chassis"/>
-        <child link="lidar_l"/>
-        <origin xyz="1.65 0.4 1" rpy="0 0 0"/>
+        <child link="camera_ray"/>
+        <origin xyz="1.65 0 1" rpy="0 0 0"/>
     </joint>
-    <link name="lidar_l">
+    <link name="camera_ray">
         <visual>
             <geometry>
                 <cylinder radius="0.05" length="0.04"/>
             </geometry>
-            <material name="red"/>
+            <material name="custom_orange10"/>
         </visual>
         <collision>
@@ -22,10 +22,15 @@
         </xacro:inertial_cylinder>
     </link>
-    <material name="red">
-        <color rgba="1 0 0 1"/>
+    <material name="custom_orange10">
+        <color rgba="1 0.55 0 1"/>
     </material>
-    <gazebo reference="lidar_l">
-        <material>Gazebo/Red</material>
-        <sensor name="lidar_l" type="ray">
+    <gazebo reference="camera_ray">
+        <material>
+            <ambient>1 0.55 0 1</ambient>
+            <diffuse>1 0.55 0 1</diffuse>
+            <specular>0.1 0.1 0.1 1</specular>
+            <emissive>0 0 0 1</emissive>
+        </material>
+        <sensor name="camera_ray" type="ray">
             <pose> 0 0 0 0 0 0 </pose>
             <visualize>true</visualize>
@@ -34,7 +39,7 @@
                 <scan>
                     <horizontal>
-                        <samples>360</samples>
-                        <min_angle>-3.14</min_angle>
-                        <max_angle>3.14</max_angle>
+                        <samples>86</samples>
+                        <min_angle>-0.75</min_angle>
+                        <max_angle>0.75</max_angle>
                     </horizontal>
                 </scan>
@@ -44,10 +49,10 @@
                 </range>
             </ray>
-            <plugin name="lidar_l_controller" filename="libgazebo_ros_ray_sensor.so">
+            <plugin name="camera_ray_controller" filename="libgazebo_ros_ray_sensor.so">
                 <ros>
                     <argument>~/out:=scan</argument>
                 </ros>
                 <output_type>sensor_msgs/LaserScan</output_type>
-                <frame_name>lidar_l</frame_name>
+                <frame_name>camera_ray</frame_name>
             </plugin>
         </sensor>

File: description/lidar_r.xacro (robot description, xacro)
@@ -41,5 +41,5 @@
                 <range>
                     <min>0.3</min>
-                    <max>12</max>
+                    <max>5</max>
                 </range>
             </ray>

File: description/robot.urdf.xacro (robot description, xacro)
@@ -17,3 +17,4 @@
     <xacro:include filename="ultrasonic_t3r2.xacro" />
     <xacro:include filename="ultrasonic_t3l2.xacro" />
+    <xacro:include filename="camera_ray.xacro" />
 </robot>
