Commit message: Moved LiDARs to 1m height and added ultrasonic sensors to the front sides of bumper doley

File: description/lidar_l.xacro (robot description, xacro)
@@ -4,5 +4,5 @@
         <parent link="chassis"/>
         <child link="lidar_l"/>
-        <origin xyz="1.65 0.4 1.175" rpy="0 0 0"/>
+        <origin xyz="1.65 0.4 1" rpy="0 0 0"/>
     </joint>
     <link name="lidar_l">

File: description/lidar_r.xacro (robot description, xacro)
@@ -4,5 +4,5 @@
         <parent link="chassis"/>
         <child link="lidar_r"/>
-        <origin xyz="1.65 -0.4 1.175" rpy="0 0 0"/>
+        <origin xyz="1.65 -0.4 1" rpy="0 0 0"/>
     </joint>
     <link name="lidar_r">

File: description/robot.urdf.xacro (robot description, xacro)
@@ -5,5 +5,5 @@
     <xacro:include filename="lidar_l.xacro" />
     <xacro:include filename="lidar_r.xacro" />
-    <!-- <xacro:include filename="ultrasonic_t1r1.xacro" /> -->
-    <!-- <xacro:include filename="ultrasonic_t1l1.xacro" /> -->
+    <xacro:include filename="ultrasonic_t1r1.xacro" />
+    <xacro:include filename="ultrasonic_t1l1.xacro" />
 </robot>

File: description/ultrasonic_t1l1.xacro (robot description, xacro)
@@ -4,5 +4,5 @@
         <parent link="cart"/>
         <child link="ultrasonic_t1l1"/>
-        <origin xyz="0.15 -0.10 0.175" rpy="0 0 -${pi/2}"/>
+        <origin xyz="-0.7 -0.65 1" rpy="0 0 -${pi/2}"/>
     </joint>
     <link name="ultrasonic_t1l1">

File: description/ultrasonic_t1r1.xacro (robot description, xacro)
@@ -4,5 +4,5 @@
         <parent link="cart"/>
         <child link="ultrasonic_t1r1"/>
-        <origin xyz="0.15 0.10 0.175" rpy="0 0 ${pi/2}"/>
+        <origin xyz="-0.7 0.65 1" rpy="0 0 ${pi/2}"/>
     </joint>
     <link name="ultrasonic_t1r1">

Commit message: Locking outdoor settings

File: description/lidar_l.xacro (robot description, xacro)
@@ -41,5 +41,5 @@
                 <range>
                     <min>0.3</min>
-                    <max>5</max>
+                    <max>12</max>
                 </range>
             </ray>

File: description/lidar_r.xacro (robot description, xacro)
@@ -41,5 +41,5 @@
                 <range>
                     <min>0.3</min>
-                    <max>5</max>
+                    <max>12</max>
                 </range>
             </ray>

File: description/robot.urdf.xacro (robot description, xacro)
@@ -5,4 +5,6 @@
     <xacro:include filename="lidar_l.xacro" />
     <xacro:include filename="lidar_r.xacro" />
+    <xacro:include filename="camera_ray.xacro" />
+    <!--
     <xacro:include filename="ultrasonic_t1r1.xacro" />
     <xacro:include filename="ultrasonic_t1l1.xacro" />
@@ -17,4 +19,4 @@
     <xacro:include filename="ultrasonic_t3r2.xacro" />
     <xacro:include filename="ultrasonic_t3l2.xacro" />
-    <xacro:include filename="camera_ray.xacro" />
+    -->
 </robot>

File: description/robot_core.xacro (robot description, xacro)
@@ -46,5 +46,5 @@
         <parent link="base_link"/>
         <child link="left_wheel"/>
-        <origin xyz="0 0.4 0" rpy="-${pi/2} 0 0"/>
+        <origin xyz="0 0.5 0" rpy="-${pi/2} 0 0"/>
         <axis xyz="0 0 1"/>
     </joint>
@@ -72,5 +72,5 @@
         <parent link="base_link"/>
         <child link="right_wheel"/>
-        <origin xyz="0 -0.4 0" rpy="${pi/2} 0 0"/>
+        <origin xyz="0 -0.5 0" rpy="${pi/2} 0 0"/>
         <axis xyz="0 0 -1"/>
     </joint>
@@ -151,5 +151,5 @@
         <parent link="cart"/>
         <child link="cart_left_wheel"/>
-        <origin xyz="2.2 0.6 0" rpy="-${pi/2} 0 0"/>
+        <origin xyz="2.2 0.8 0" rpy="-${pi/2} 0 0"/>
         <axis xyz="0 0 1"/>
     </joint>
@@ -177,5 +177,5 @@
         <parent link="cart"/>
         <child link="cart_right_wheel"/>
-        <origin xyz="2.2 -0.6 0" rpy="${pi/2} 0 0"/>
+        <origin xyz="2.2 -0.8 0" rpy="${pi/2} 0 0"/>
         <axis xyz="0 0 -1"/>
     </joint>
@@ -229,5 +229,5 @@
         <parent link="cart2"/>
         <child link="cart2_left_wheel"/>
-        <origin xyz="1.6 0.55 0" rpy="-${pi/2} 0 0"/>
+        <origin xyz="1.6 0.7 0" rpy="-${pi/2} 0 0"/>
         <axis xyz="0 0 1"/>
     </joint>
@@ -254,5 +254,5 @@
         <parent link="cart2"/>
         <child link="cart2_right_wheel"/>
-        <origin xyz="1.6 -0.55 0" rpy="${pi/2} 0 0"/>
+        <origin xyz="1.6 -0.7 0" rpy="${pi/2} 0 0"/>
         <axis xyz="0 0 -1"/>
     </joint>
