Commit message: <Progress on Launch issue> Modified ros2_control to make things work better with Gazebo 11. Loading controller fails but at least command and state interfaces load.

File: description/ros2_control.xacro (robot description, xacro)
@@ -2,28 +2,20 @@
 <robot xmlns:xacro="http://www.ros.org/wiki/xacro">
     <ros2_control name="GazeboSystem" type="system">
-        <hardware>
-            <plugin>gazebo_ros2_control/GazeboSystem</plugin>
-        </hardware>
-        <joint name="left_wheel_joint">
-            <command_interface name="velocity">
-                <param name="min">-10</param>
-                <param name="max">10</param>
-            </command_interface>
-            <state_interface name="velocity"/>
-            <state_interface name="position"/>
-        </joint>
-        <joint name="right_wheel_joint">
-            <command_interface name="velocity">
-                <param name="min">-10</param>
-                <param name="max">10</param>
-            </command_interface>
-            <state_interface name="velocity"/>
-            <state_interface name="position"/>
-        </joint>
+    <hardware>
+        <plugin>gazebo_ros2_control/GazeboSystem</plugin>
+    </hardware>
+    <joint name="left_wheel_joint">
+        <command_interface name="velocity"/>
+        <state_interface name="velocity"/>
+    </joint>
+    <joint name="right_wheel_joint">
+        <command_interface name="velocity"/>
+        <state_interface name="velocity"/>
+    </joint>
     </ros2_control>
     <gazebo>
-        <plugin name='gazebo_ros2_control' filename='libgazebo_ros2_control.so'>
-            <parameters>$(find diff_drive_robot)/config/my_controllers.yaml</parameters>
-        </plugin>
+    <plugin name="gazebo_ros2_control" filename="libgazebo_ros2_control.so">
+        <parameters>$(find diff_drive_robot)/config/my_controllers.yaml</parameters>
+    </plugin>
     </gazebo>
 </robot>
