Commit message: Renamed lidar link from "laser_frame" to "lidar"

File: description/lidar.xacro (robot description, xacro)
@@ -1,10 +1,10 @@
 <?xml version="1.0"?>
 <robot xmlns:xacro="http://www.ros.org/wiki/xacro" >
-    <joint name="laser_joint" type="fixed">
+    <joint name="lidar_joint" type="fixed">
         <parent link="chassis"/>
-        <child link="laser_frame"/>
+        <child link="lidar"/>
         <origin xyz="0.1 0 0.175" rpy="0 0 0"/>
     </joint>
-    <link name="laser_frame">
+    <link name="lidar">
         ...fill in here...
     </link>

Commit message: Defined the lidar visual, collision, inertia, and color

File: description/lidar.xacro (robot description, xacro)
@@ -7,5 +7,22 @@
     </joint>
     <link name="lidar">
-        ...fill in here...
+        <visual>
+            <geometry>
+                <cylinder radius="0.05" length="0.04"/>
+            </geometry>
+            <material name="red"/>
+        </visual>
+        <collision>
+            <geometry>
+                <cylinder radius="0.05" length="0.04"/>
+            </geometry>
+        </collision>
+        <xacro:inertial_cylinder mass="0.1" length="0.04" radius="0.05">
+            <origin xyz="0 0 0" rpy="0 0 0"/>
+        </xacro:inertial_cylinder>
     </link>
+    <gazebo reference="lidar">
+        <material>Gazebo/Red</material>
+        ... Yet to put stuff here ...
+    </gazebo>
 </robot>

File: description/robot_core.xacro (robot description, xacro)
@@ -7,4 +7,7 @@
     <material name="orange">
         <color rgba="1 0.3 0.1 1"/>
+    </material>
+    <material name="red">
+        <color rgba="1 0 0 1"/>
     </material>
     <material name="blue">

Commit message: Moved lidar color definition from robot core file to lidar.xacro file; functionality remains unchanged

File: description/lidar.xacro (robot description, xacro)
@@ -22,4 +22,7 @@
         </xacro:inertial_cylinder>
     </link>
+    <material name="red">
+        <color rgba="1 0 0 1"/>
+    </material>
     <gazebo reference="lidar">
         <material>Gazebo/Red</material>

File: description/robot_core.xacro (robot description, xacro)
@@ -7,7 +7,4 @@
     <material name="orange">
         <color rgba="1 0.3 0.1 1"/>
-    </material>
-    <material name="red">
-        <color rgba="1 0 0 1"/>
     </material>
     <material name="blue">

Commit message: Only enabled cart 1 and limited main LiDAR range to 180 degrees in prep of fixing cart tf to map frame. Temporary tf data (temp_tf_data_comparison.txt) showcasing missing transforms added to package directory

File: description/lidar.xacro (robot description, xacro)
@@ -35,6 +35,6 @@
                     <horizontal>
                         <samples>360</samples>
-                        <min_angle>-3.14</min_angle>
-                        <max_angle>3.14</max_angle>
+                        <min_angle>-1.57</min_angle>
+                        <max_angle>1.57</max_angle>
                     </horizontal>
                 </scan>

File: description/robot_core.xacro (robot description, xacro)
@@ -207,5 +207,5 @@
     </gazebo>
     <!-- CART 2 -->
-    <joint name="cart2_joint" type="revolute">
+    <!-- <joint name="cart2_joint" type="revolute">
         <parent link="cart"/>
         <child link="cart2"/>
@@ -231,7 +231,7 @@
             <origin xyz="0.15 0 0.075" rpy="0 0 0"/>
         </xacro:inertial_box>
-    </link>
+    </link> -->
     <!-- LEFT WHEEL -->
-    <joint name="cart2_left_wheel_joint" type="continuous">
+    <!-- <joint name="cart2_left_wheel_joint" type="continuous">
         <parent link="cart2"/>
         <child link="cart2_left_wheel"/>
@@ -257,7 +257,7 @@
     <gazebo reference="cart2_left_wheel">
         <material>Gazebo/Blue</material>
-    </gazebo>
+    </gazebo> -->
     <!-- RIGHT WHEEL -->
-    <joint name="cart2_right_wheel_joint" type="continuous">
+    <!-- <joint name="cart2_right_wheel_joint" type="continuous">
         <parent link="cart2"/>
         <child link="cart2_right_wheel"/>
@@ -283,4 +283,4 @@
     <gazebo reference="cart2_right_wheel">
         <material>Gazebo/Blue</material>
-    </gazebo>
+    </gazebo> -->
 </robot>
