Commit message: Added collision

File: description/robot_core.xacro (robot description, xacro)
@@ -28,4 +28,10 @@
             <material name="white"/>
         </visual>
+        <collision>
+            <origin xyz="0.15 0 0.075" rpy="0 0 0"/>
+            <geometry>
+                <box size="0.3 0.3 0.15"/>
+            </geometry>
+        </collision>
     </link>
     <!-- LEFT WHEEL -->
@@ -43,4 +49,9 @@
             <material name="blue"/>
         </visual>
+        <collision>
+            <geometry>
+                <cylinder length="0.04" radius="0.05" />
+            </geometry>
+        </collision>
     </link>
     <!-- RIGHT WHEEL -->
@@ -58,4 +69,9 @@
             <material name="blue"/>
         </visual>
+        <collision>
+            <geometry>
+                <cylinder length="0.04" radius="0.05" />
+            </geometry>
+        </collision>
     </link>
     <!-- CASTER WHEEL -->
@@ -72,4 +88,9 @@
             <material name="black"/>
         </visual>
+        <collision>
+            <geometry>
+                <cylinder length="0.04" radius="0.05" />
+            </geometry>
+        </collision>
     </link>
 </robot>

Commit message: Added inertial macros to all links

File: description/robot_core.xacro (robot description, xacro)
@@ -1,4 +1,5 @@
 <?xml version="1.0"?>
 <robot xmlns:xacro="http://www.ros.org/wiki/xacro">
+    <xacro:include filename="inertial_macros.xacro" />
     <material name="white">
         <color rgba="1 1 1 1"/>
@@ -34,4 +35,7 @@
             </geometry>
         </collision>
+        <xacro:inertial_box mass="0.5" x="0.3" y="0.3" z="0.15">
+            <origin xyz="0.15 0 0.075" rpy="0 0 0"/>
+        </xacro:inertial_box>
     </link>
     <!-- LEFT WHEEL -->
@@ -54,4 +58,7 @@
             </geometry>
         </collision>
+        <xacro:inertial_cylinder mass="0.1" length="0.05" radius="0.05">
+            <origin xyz="0 0 0" rpy="0 0 0"/>
+        </xacro:inertial_cylinder>
     </link>
     <!-- RIGHT WHEEL -->
@@ -74,4 +81,7 @@
             </geometry>
         </collision>
+        <xacro:inertial_cylinder mass="0.1" length="0.05" radius="0.05">
+            <origin xyz="0 0 0" rpy="0 0 0"/>
+        </xacro:inertial_cylinder>
     </link>
     <!-- CASTER WHEEL -->
@@ -93,4 +103,7 @@
             </geometry>
         </collision>
+        <xacro:inertial_sphere mass="0.1" radius="0.05">
+            <origin xyz="0 0 0" rpy="0 0 0"/>
+        </xacro:inertial_sphere>
     </link>
 </robot>

Commit message: Added colors to Gazebo simulation robot

File: description/robot_core.xacro (robot description, xacro)
@@ -39,4 +39,7 @@
         </xacro:inertial_box>
     </link>
+    <gazebo reference="chassis">
+        <material>Gazebo/White</material>
+    </gazebo>
     <!-- LEFT WHEEL -->
     <joint name="left_wheel_joint" type="continuous">
@@ -62,4 +65,7 @@
         </xacro:inertial_cylinder>
     </link>
+    <gazebo reference="left_wheel">
+        <material>Gazebo/Blue</material>
+    </gazebo>
     <!-- RIGHT WHEEL -->
     <joint name="right_wheel_joint" type="continuous">
@@ -85,4 +91,7 @@
         </xacro:inertial_cylinder>
     </link>
+    <gazebo reference="right_wheel">
+        <material>Gazebo/Blue</material>
+    </gazebo>
     <!-- CASTER WHEEL -->
     <joint name="caster_wheel_joint" type="fixed">
@@ -107,3 +116,6 @@
         </xacro:inertial_sphere>
     </link>
+    <gazebo reference="caster_wheel">
+        <material>Gazebo/Black</material>
+    </gazebo>
 </robot>

Commit message: Fixed robot tilt by adding z offset to caster wheel joint

File: description/robot_core.xacro (robot description, xacro)
@@ -98,5 +98,5 @@
         <parent link="chassis"/>
         <child link="caster_wheel"/>
-        <origin xyz="0.24 0 0" rpy="0 0 0"/>
+        <origin xyz="0.24 0 -0.03" rpy="0 0 0"/>
     </joint>
     <link name="caster_wheel">

Commit message: Added a cart (without wheels) behind the robot through a revolute joint

File: description/robot_core.xacro (robot description, xacro)
@@ -42,4 +42,30 @@
         <material>Gazebo/White</material>
     </gazebo>
+    <!-- CART -->
+    <joint name="cart_joint" type="revolute">
+        <parent link="chassis"/>
+        <child link="cart"/>
+        <origin xyz="-0.15 0 0" rpy="0 0 ${pi}"/>
+        <axis xyz="0 0 1"/>
+        <limit effort="10" velocity="1.0" lower="-1.57" upper="1.57"/>
+    </joint>
+    <link name="cart">
+        <visual>
+            <origin xyz="0.15 0 0.075" rpy="0 0 0"/>
+            <geometry>
+                <box size="0.3 0.3 0.15"/>
+            </geometry>
+            <material name="white"/>
+        </visual>
+        <collision>
+            <origin xyz="0.15 0 0.075" rpy="0 0 0"/>
+            <geometry>
+                <box size="0.3 0.3 0.15"/>
+            </geometry>
+        </collision>
+        <xacro:inertial_box mass="0.5" x="0.3" y="0.3" z="0.15">
+            <origin xyz="0.15 0 0.075" rpy="0 0 0"/>
+        </xacro:inertial_box>
+    </link>
     <!-- LEFT WHEEL -->
     <joint name="left_wheel_joint" type="continuous">

Commit message: Added wheels to the cart; simulation matches reality reasonably well. Tow Truck and Trailer System V1 complete.

File: description/robot_core.xacro (robot description, xacro)
@@ -41,4 +41,83 @@
     <gazebo reference="chassis">
         <material>Gazebo/White</material>
+    </gazebo>
+    <!-- LEFT WHEEL -->
+    <joint name="left_wheel_joint" type="continuous">
+        <parent link="base_link"/>
+        <child link="left_wheel"/>
+        <origin xyz="0 0.175 0" rpy="-${pi/2} 0 0"/>
+        <axis xyz="0 0 1"/>
+    </joint>
+    <link name="left_wheel">
+        <visual>
+            <geometry>
+                <cylinder length="0.04" radius="0.05" />
+            </geometry>
+            <material name="blue"/>
+        </visual>
+        <collision>
+            <geometry>
+                <cylinder length="0.04" radius="0.05" />
+            </geometry>
+        </collision>
+        <xacro:inertial_cylinder mass="0.1" length="0.05" radius="0.05">
+            <origin xyz="0 0 0" rpy="0 0 0"/>
+        </xacro:inertial_cylinder>
+    </link>
+    <gazebo reference="left_wheel">
+        <material>Gazebo/Blue</material>
+    </gazebo>
+    <!-- RIGHT WHEEL -->
+    <joint name="right_wheel_joint" type="continuous">
+        <parent link="base_link"/>
+        <child link="right_wheel"/>
+        <origin xyz="0 -0.175 0" rpy="${pi/2} 0 0"/>
+        <axis xyz="0 0 -1"/>
+    </joint>
+    <link name="right_wheel">
+        <visual>
+            <geometry>
+                <cylinder length="0.04" radius="0.05" />
+            </geometry>
+            <material name="blue"/>
+        </visual>
+        <collision>
+            <geometry>
+                <cylinder length="0.04" radius="0.05" />
+            </geometry>
+        </collision>
+        <xacro:inertial_cylinder mass="0.1" length="0.05" radius="0.05">
+            <origin xyz="0 0 0" rpy="0 0 0"/>
+        </xacro:inertial_cylinder>
+    </link>
+    <gazebo reference="right_wheel">
+        <material>Gazebo/Blue</material>
+    </gazebo>
+    <!-- CASTER WHEEL -->
+    <joint name="caster_wheel_joint" type="fixed">
+        <parent link="chassis"/>
+        <child link="caster_wheel"/>
+        <origin xyz="0.24 0 -0.03" rpy="0 0 0"/>
+    </joint>
+    <link name="caster_wheel">
+        <visual>
+            <geometry>
+                <sphere radius="0.05" />
+            </geometry>
+            <material name="black"/>
+        </visual>
+        <collision>
+            <geometry>
+                <cylinder length="0.04" radius="0.05" />
+            </geometry>
+        </collision>
+        <xacro:inertial_sphere mass="0.1" radius="0.05">
+            <origin xyz="0 0 0" rpy="0 0 0"/>
+        </xacro:inertial_sphere>
+    </link>
+    <gazebo reference="caster_wheel">
+        <material>Gazebo/Black</material>
+        <mu1 value="0.5"/>
+        <mu2 value="0.5"/>
     </gazebo>
     <!-- CART -->
@@ -69,81 +148,54 @@
     </link>
     <!-- LEFT WHEEL -->
-    <joint name="left_wheel_joint" type="continuous">
-        <parent link="base_link"/>
-        <child link="left_wheel"/>
-        <origin xyz="0 0.175 0" rpy="-${pi/2} 0 0"/>
+    <joint name="cart_left_wheel_joint" type="continuous">
+        <parent link="cart"/>
+        <child link="cart_left_wheel"/>
+        <origin xyz="0.28 0.175 0" rpy="-${pi/2} 0 0"/>
         <axis xyz="0 0 1"/>
     </joint>
-    <link name="left_wheel">
-        <visual>
-            <geometry>
-                <cylinder length="0.04" radius="0.05" />
-            </geometry>
-            <material name="blue"/>
-        </visual>
-        <collision>
-            <geometry>
-                <cylinder length="0.04" radius="0.05" />
-            </geometry>
-        </collision>
-        <xacro:inertial_cylinder mass="0.1" length="0.05" radius="0.05">
-            <origin xyz="0 0 0" rpy="0 0 0"/>
-        </xacro:inertial_cylinder>
-    </link>
-    <gazebo reference="left_wheel">
+    <link name="cart_left_wheel">
+        <visual>
+            <geometry>
+                <cylinder length="0.04" radius="0.05" />
+            </geometry>
+            <material name="blue"/>
+        </visual>
+        <collision>
+            <geometry>
+                <cylinder length="0.04" radius="0.05" />
+            </geometry>
+        </collision>
+        <xacro:inertial_cylinder mass="0.1" length="0.05" radius="0.05">
+            <origin xyz="0 0 0" rpy="0 0 0"/>
+        </xacro:inertial_cylinder>
+    </link>
+    <gazebo reference="cart_left_wheel">
         <material>Gazebo/Blue</material>
     </gazebo>
     <!-- RIGHT WHEEL -->
-    <joint name="right_wheel_joint" type="continuous">
-        <parent link="base_link"/>
-        <child link="right_wheel"/>
-        <origin xyz="0 -0.175 0" rpy="${pi/2} 0 0"/>
+    <joint name="cart_right_wheel_joint" type="continuous">
+        <parent link="cart"/>
+        <child link="cart_right_wheel"/>
+        <origin xyz="0.28 -0.175 0" rpy="${pi/2} 0 0"/>
         <axis xyz="0 0 -1"/>
     </joint>
-    <link name="right_wheel">
-        <visual>
-            <geometry>
-                <cylinder length="0.04" radius="0.05" />
-            </geometry>
-            <material name="blue"/>
-        </visual>
-        <collision>
-            <geometry>
-                <cylinder length="0.04" radius="0.05" />
-            </geometry>
-        </collision>
-        <xacro:inertial_cylinder mass="0.1" length="0.05" radius="0.05">
-            <origin xyz="0 0 0" rpy="0 0 0"/>
-        </xacro:inertial_cylinder>
-    </link>
-    <gazebo reference="right_wheel">
-        <material>Gazebo/Blue</material>
-    </gazebo>
-    <!-- CASTER WHEEL -->
-    <joint name="caster_wheel_joint" type="fixed">
-        <parent link="chassis"/>
-        <child link="caster_wheel"/>
-        <origin xyz="0.24 0 -0.03" rpy="0 0 0"/>
-    </joint>
-    <link name="caster_wheel">
-        <visual>
-            <geometry>
-                <sphere radius="0.05" />
-            </geometry>
-            <material name="black"/>
-        </visual>
-        <collision>
-            <geometry>
-                <cylinder length="0.04" radius="0.05" />
-            </geometry>
-        </collision>
-        <xacro:inertial_sphere mass="0.1" radius="0.05">
-            <origin xyz="0 0 0" rpy="0 0 0"/>
-        </xacro:inertial_sphere>
-    </link>
-    <gazebo reference="caster_wheel">
-        <material>Gazebo/Black</material>
-        <mu1 value="0.5"/>
-        <mu2 value="0.5"/>
+    <link name="cart_right_wheel">
+        <visual>
+            <geometry>
+                <cylinder length="0.04" radius="0.05" />
+            </geometry>
+            <material name="blue"/>
+        </visual>
+        <collision>
+            <geometry>
+                <cylinder length="0.04" radius="0.05" />
+            </geometry>
+        </collision>
+        <xacro:inertial_cylinder mass="0.1" length="0.05" radius="0.05">
+            <origin xyz="0 0 0" rpy="0 0 0"/>
+        </xacro:inertial_cylinder>
+    </link>
+    <gazebo reference="cart_right_wheel">
+        <material>Gazebo/Blue</material>
     </gazebo>
 </robot>

Commit message: Added a second cart. Tow Truck and Trailer System v2 complete.

File: description/robot_core.xacro (robot description, xacro)
@@ -199,3 +199,81 @@
         <material>Gazebo/Blue</material>
     </gazebo>
+<!-- CART 2 -->
+    <joint name="cart2_joint" type="revolute">
+        <parent link="cart"/>
+        <child link="cart2"/>
+        <origin xyz="0.45 0 0" rpy="0 0 0"/>
+        <axis xyz="0 0 1"/>
+        <limit effort="10" velocity="1.0" lower="-1.57" upper="1.57"/>
+    </joint>
+    <link name="cart2">
+        <visual>
+            <origin xyz="0.15 0 0.075" rpy="0 0 0"/>
+            <geometry>
+                <box size="0.3 0.3 0.15"/>
+            </geometry>
+            <material name="white"/>
+        </visual>
+        <collision>
+            <origin xyz="0.15 0 0.075" rpy="0 0 0"/>
+            <geometry>
+                <box size="0.3 0.3 0.15"/>
+            </geometry>
+        </collision>
+        <xacro:inertial_box mass="0.5" x="0.3" y="0.3" z="0.15">
+            <origin xyz="0.15 0 0.075" rpy="0 0 0"/>
+        </xacro:inertial_box>
+    </link>
+    <!-- LEFT WHEEL -->
+    <joint name="cart2_left_wheel_joint" type="continuous">
+        <parent link="cart2"/>
+        <child link="cart2_left_wheel"/>
+        <origin xyz="0.28 0.175 0" rpy="-${pi/2} 0 0"/>
+        <axis xyz="0 0 1"/>
+    </joint>
+    <link name="cart2_left_wheel">
+        <visual>
+            <geometry>
+                <cylinder length="0.04" radius="0.05" />
+            </geometry>
+            <material name="blue"/>
+        </visual>
+        <collision>
+            <geometry>
+                <cylinder length="0.04" radius="0.05" />
+            </geometry>
+        </collision>
+        <xacro:inertial_cylinder mass="0.1" length="0.05" radius="0.05">
+            <origin xyz="0 0 0" rpy="0 0 0"/>
+        </xacro:inertial_cylinder>
+    </link>
+    <gazebo reference="cart2_left_wheel">
+        <material>Gazebo/Blue</material>
+    </gazebo>
+    <!-- RIGHT WHEEL -->
+    <joint name="cart2_right_wheel_joint" type="continuous">
+        <parent link="cart2"/>
+        <child link="cart2_right_wheel"/>
+        <origin xyz="0.28 -0.175 0" rpy="${pi/2} 0 0"/>
+        <axis xyz="0 0 -1"/>
+    </joint>
+    <link name="cart2_right_wheel">
+        <visual>
+            <geometry>
+                <cylinder length="0.04" radius="0.05" />
+            </geometry>
+            <material name="blue"/>
+        </visual>
+        <collision>
+            <geometry>
+                <cylinder length="0.04" radius="0.05" />
+            </geometry>
+        </collision>
+        <xacro:inertial_cylinder mass="0.1" length="0.05" radius="0.05">
+            <origin xyz="0 0 0" rpy="0 0 0"/>
+        </xacro:inertial_cylinder>
+    </link>
+    <gazebo reference="cart2_right_wheel">
+        <material>Gazebo/Blue</material>
+    </gazebo>
 </robot>

Commit message: Modelled differential drive tow truck at full scale

File: description/robot_core.xacro (robot description, xacro)
@@ -23,18 +23,18 @@
     <link name="chassis">
         <visual>
-            <origin xyz="0.8225 0 1.0" rpy="0 0 0"/>
-            <geometry>
-                <box size="1.645 0.8 2"/>
+            <origin xyz="0.8225 0 0.85" rpy="0 0 0"/>
+            <geometry>
+                <box size="1.645 0.8 1.8"/>
             </geometry>
             <material name="white"/>
         </visual>
         <collision>
-            <origin xyz="0.8225 0 1.0" rpy="0 0 0"/>
-            <geometry>
-                <box size="1.645 0.8 2"/>
-            </geometry>
-        </collision>
-        <xacro:inertial_box mass="50" x="1.645" y="0.8" z="2">
-            <origin xyz="0.8225 0 1.0" rpy="0 0 0"/>
+            <origin xyz="0.8225 0 0.85" rpy="0 0 0"/>
+            <geometry>
+                <box size="1.645 0.8 1.8"/>
+            </geometry>
+        </collision>
+        <xacro:inertial_box mass="100" x="1.645" y="0.8" z="1.8">
+            <origin xyz="0.8225 0 0.85" rpy="0 0 0"/>
         </xacro:inertial_box>
     </link>
@@ -46,5 +46,5 @@
         <parent link="base_link"/>
         <child link="left_wheel"/>
-        <origin xyz="0 0.4 0.2" rpy="-${pi/2} 0 0"/>
+        <origin xyz="0 0.4 0" rpy="-${pi/2} 0 0"/>
         <axis xyz="0 0 1"/>
     </joint>
@@ -61,5 +61,5 @@
             </geometry>
         </collision>
-        <xacro:inertial_cylinder mass="5" length="0.1" radius="0.2">
+        <xacro:inertial_cylinder mass="10" length="0.1" radius="0.2">
             <origin xyz="0 0 0" rpy="0 0 0"/>
         </xacro:inertial_cylinder>
@@ -72,5 +72,5 @@
         <parent link="base_link"/>
         <child link="right_wheel"/>
-        <origin xyz="0 -0.4 0.2" rpy="${pi/2} 0 0"/>
+        <origin xyz="0 -0.4 0" rpy="${pi/2} 0 0"/>
         <axis xyz="0 0 -1"/>
     </joint>
@@ -87,5 +87,5 @@
             </geometry>
         </collision>
-        <xacro:inertial_cylinder mass="5" length="0.1" radius="0.2">
+        <xacro:inertial_cylinder mass="10" length="0.1" radius="0.2">
             <origin xyz="0 0 0" rpy="0 0 0"/>
         </xacro:inertial_cylinder>
@@ -98,5 +98,5 @@
         <parent link="chassis"/>
         <child link="caster_wheel"/>
-        <origin xyz="1.2 0 -0.1" rpy="0 0 0"/>
+        <origin xyz="1.4 0 -0.1" rpy="0 0 0"/>
     </joint>
     <link name="caster_wheel">
@@ -112,5 +112,5 @@
             </geometry>
         </collision>
-        <xacro:inertial_sphere mass="2" radius="0.1">
+        <xacro:inertial_sphere mass="10" radius="0.1">
             <origin xyz="0 0 0" rpy="0 0 0"/>
         </xacro:inertial_sphere>
@@ -118,6 +118,6 @@
     <gazebo reference="caster_wheel">
         <material>Gazebo/Black</material>
-        <mu1 value="0.5"/>
-        <mu2 value="0.5"/>
+        <mu1 value="0.15"/>
+        <mu2 value="0.15"/>
     </gazebo>
     <!--

Commit message: Added full-scale grill doley 1

File: description/robot_core.xacro (robot description, xacro)
@@ -121,9 +121,9 @@
         <mu2 value="0.15"/>
     </gazebo>
-    <!--
+    <!-- Cart -->
     <joint name="cart_joint" type="revolute">
         <parent link="chassis"/>
         <child link="cart"/>
-        <origin xyz="-0.15 0 0" rpy="0 0 ${pi}"/>
+        <origin xyz="-0.5334 0 0" rpy="0 0 ${pi}"/>
         <axis xyz="0 0 1"/>
         <limit effort="10" velocity="1.0" lower="-1.57" upper="1.57"/>
@@ -131,24 +131,25 @@
     <link name="cart">
         <visual>
-            <origin xyz="0.15 0 0.075" rpy="0 0 0"/>
-            <geometry>
-                <box size="0.3 0.3 0.15"/>
+            <origin xyz="0.9 0 1.12" rpy="0 0 0"/>
+            <geometry>
+                <box size="1.8 1.11 2.24"/>
             </geometry>
             <material name="white"/>
         </visual>
         <collision>
-            <origin xyz="0.15 0 0.075" rpy="0 0 0"/>
-            <geometry>
-                <box size="0.3 0.3 0.15"/>
-            </geometry>
-        </collision>
-        <xacro:inertial_box mass="0.5" x="0.3" y="0.3" z="0.15">
-            <origin xyz="0.15 0 0.075" rpy="0 0 0"/>
+            <origin xyz="0.9 0 1.12" rpy="0 0 0"/>
+            <geometry>
+                <box size="1.8 1.11 2.24"/>
+            </geometry>
+        </collision>
+        <xacro:inertial_box mass="200" x="1.8" y="1.11" z="2.24">
+            <origin xyz="0.9 0 1.12" rpy="0 0 0"/>
         </xacro:inertial_box>
     </link>
+    <!-- Cart Left Wheel -->
     <joint name="cart_left_wheel_joint" type="continuous">
         <parent link="cart"/>
         <child link="cart_left_wheel"/>
-        <origin xyz="0.28 0.175 0" rpy="-${pi/2} 0 0"/>
+        <origin xyz="1.6 0.55 0" rpy="-${pi/2} 0 0"/>
         <axis xyz="0 0 1"/>
     </joint>
@@ -156,14 +157,14 @@
         <visual>
             <geometry>
-                <cylinder length="0.04" radius="0.05" />
-            </geometry>
-            <material name="blue"/>
-        </visual>
-        <collision>
-            <geometry>
-                <cylinder length="0.04" radius="0.05" />
-            </geometry>
-        </collision>
-        <xacro:inertial_cylinder mass="0.1" length="0.05" radius="0.05">
+                <cylinder length="0.2" radius="0.15" />
+            </geometry>
+            <material name="blue"/>
+        </visual>
+        <collision>
+            <geometry>
+                <cylinder length="0.2" radius="0.15" />
+            </geometry>
+        </collision>
+        <xacro:inertial_cylinder mass="5" length="0.2" radius="0.15">
             <origin xyz="0 0 0" rpy="0 0 0"/>
         </xacro:inertial_cylinder>
@@ -172,8 +173,9 @@
         <material>Gazebo/Blue</material>
     </gazebo>
+    <!-- Cart Right Wheel -->
     <joint name="cart_right_wheel_joint" type="continuous">
         <parent link="cart"/>
         <child link="cart_right_wheel"/>
-        <origin xyz="0.28 -0.175 0" rpy="${pi/2} 0 0"/>
+        <origin xyz="1.6 -0.55 0" rpy="${pi/2} 0 0"/>
         <axis xyz="0 0 -1"/>
     </joint>
@@ -181,14 +183,14 @@
         <visual>
             <geometry>
-                <cylinder length="0.04" radius="0.05" />
-            </geometry>
-            <material name="blue"/>
-        </visual>
-        <collision>
-            <geometry>
-                <cylinder length="0.04" radius="0.05" />
-            </geometry>
-        </collision>
-        <xacro:inertial_cylinder mass="0.1" length="0.05" radius="0.05">
+                <cylinder length="0.2" radius="0.15" />
+            </geometry>
+            <material name="blue"/>
+        </visual>
+        <collision>
+            <geometry>
+                <cylinder length="0.2" radius="0.15" />
+            </geometry>
+        </collision>
+        <xacro:inertial_cylinder mass="5" length="0.2" radius="0.15">
             <origin xyz="0 0 0" rpy="0 0 0"/>
         </xacro:inertial_cylinder>
@@ -197,4 +199,5 @@
         <material>Gazebo/Blue</material>
     </gazebo>
+    <!--
     <joint name="cart2_joint" type="revolute">
         <parent link="cart"/>
