Commit message: Added full-scale grill doley 2 (cart 2); Broke physics

File: description/robot_core.xacro (robot description, xacro)
@@ -199,9 +199,9 @@
         <material>Gazebo/Blue</material>
     </gazebo>
-    <!--
+    <!-- Cart 2 -->
     <joint name="cart2_joint" type="revolute">
         <parent link="cart"/>
         <child link="cart2"/>
-        <origin xyz="0.45 0 0" rpy="0 0 0"/>
+        <origin xyz="2.3334 0 0" rpy="0 0 0"/>
         <axis xyz="0 0 1"/>
         <limit effort="10" velocity="1.0" lower="-1.57" upper="1.57"/>
@@ -209,18 +209,18 @@
     <link name="cart2">
         <visual>
-            <origin xyz="0.15 0 0.075" rpy="0 0 0"/>
-            <geometry>
-                <box size="0.3 0.3 0.15"/>
+            <origin xyz="0.9 0 1.12" rpy="0 0 0"/>
+            <geometry>
+                <box size="1.8 1.11 2.24"/>
             </geometry>
             <material name="white"/>
         </visual>
         <collision>
-            <origin xyz="0.15 0 0.075" rpy="0 0 0"/>
-            <geometry>
-                <box size="0.3 0.3 0.15"/>
-            </geometry>
-        </collision>
-        <xacro:inertial_box mass="0.5" x="0.3" y="0.3" z="0.15">
-            <origin xyz="0.15 0 0.075" rpy="0 0 0"/>
+            <origin xyz="0.9 0 1.12" rpy="0 0 0"/>
+            <geometry>
+                <box size="1.8 1.11 2.24"/>
+            </geometry>
+        </collision>
+        <xacro:inertial_box mass="200" x="1.8" y="1.11" z="2.24">
+            <origin xyz="0.9 0 1.12" rpy="0 0 0"/>
         </xacro:inertial_box>
     </link>
@@ -228,5 +228,5 @@
         <parent link="cart2"/>
         <child link="cart2_left_wheel"/>
-        <origin xyz="0.28 0.175 0" rpy="-${pi/2} 0 0"/>
+        <origin xyz="1.6 0.55 0" rpy="-${pi/2} 0 0"/>
         <axis xyz="0 0 1"/>
     </joint>
@@ -234,14 +234,14 @@
         <visual>
             <geometry>
-                <cylinder length="0.04" radius="0.05" />
-            </geometry>
-            <material name="blue"/>
-        </visual>
-        <collision>
-            <geometry>
-                <cylinder length="0.04" radius="0.05" />
-            </geometry>
-        </collision>
-        <xacro:inertial_cylinder mass="0.1" length="0.05" radius="0.05">
+                <cylinder length="0.2" radius="0.15" />
+            </geometry>
+            <material name="blue"/>
+        </visual>
+        <collision>
+            <geometry>
+                <cylinder length="0.2" radius="0.15" />
+            </geometry>
+        </collision>
+        <xacro:inertial_cylinder mass="5" length="0.2" radius="0.15">
             <origin xyz="0 0 0" rpy="0 0 0"/>
         </xacro:inertial_cylinder>
@@ -253,5 +253,5 @@
         <parent link="cart2"/>
         <child link="cart2_right_wheel"/>
-        <origin xyz="0.28 -0.175 0" rpy="${pi/2} 0 0"/>
+        <origin xyz="1.6 -0.55 0" rpy="${pi/2} 0 0"/>
         <axis xyz="0 0 -1"/>
     </joint>
@@ -259,14 +259,14 @@
         <visual>
             <geometry>
-                <cylinder length="0.04" radius="0.05" />
-            </geometry>
-            <material name="blue"/>
-        </visual>
-        <collision>
-            <geometry>
-                <cylinder length="0.04" radius="0.05" />
-            </geometry>
-        </collision>
-        <xacro:inertial_cylinder mass="0.1" length="0.05" radius="0.05">
+                <cylinder length="0.2" radius="0.15" />
+            </geometry>
+            <material name="blue"/>
+        </visual>
+        <collision>
+            <geometry>
+                <cylinder length="0.2" radius="0.15" />
+            </geometry>
+        </collision>
+        <xacro:inertial_cylinder mass="5" length="0.2" radius="0.15">
             <origin xyz="0 0 0" rpy="0 0 0"/>
         </xacro:inertial_cylinder>
@@ -275,4 +275,3 @@
         <material>Gazebo/Blue</material>
     </gazebo>
-    -->
 </robot>

Commit message: Trial 1 of fixing physics: changed masses, cart sizes, hitch 2 length; physics is still broken

File: description/robot_core.xacro (robot description, xacro)
@@ -35,5 +35,5 @@
             </geometry>
         </collision>
-        <xacro:inertial_box mass="100" x="1.645" y="0.8" z="1.8">
+        <xacro:inertial_box mass="50" x="1.645" y="0.8" z="1.8">
             <origin xyz="0.8225 0 0.85" rpy="0 0 0"/>
         </xacro:inertial_box>
@@ -61,5 +61,5 @@
             </geometry>
         </collision>
-        <xacro:inertial_cylinder mass="10" length="0.1" radius="0.2">
+        <xacro:inertial_cylinder mass="5" length="0.1" radius="0.2">
             <origin xyz="0 0 0" rpy="0 0 0"/>
         </xacro:inertial_cylinder>
@@ -87,5 +87,5 @@
             </geometry>
         </collision>
-        <xacro:inertial_cylinder mass="10" length="0.1" radius="0.2">
+        <xacro:inertial_cylinder mass="5" length="0.1" radius="0.2">
             <origin xyz="0 0 0" rpy="0 0 0"/>
         </xacro:inertial_cylinder>
@@ -112,5 +112,5 @@
             </geometry>
         </collision>
-        <xacro:inertial_sphere mass="10" radius="0.1">
+        <xacro:inertial_sphere mass="5" radius="0.1">
             <origin xyz="0 0 0" rpy="0 0 0"/>
         </xacro:inertial_sphere>
@@ -131,17 +131,17 @@
     <link name="cart">
         <visual>
+            <origin xyz="0.9 0 0.7" rpy="0 0 0"/>
+            <geometry>
+                <box size="1.8 1.11 1.5"/>
+            </geometry>
+            <material name="white"/>
+        </visual>
+        <collision>
             <origin xyz="0.9 0 1.12" rpy="0 0 0"/>
             <geometry>
                 <box size="1.8 1.11 2.24"/>
             </geometry>
-            <material name="white"/>
-        </visual>
-        <collision>
-            <origin xyz="0.9 0 1.12" rpy="0 0 0"/>
-            <geometry>
-                <box size="1.8 1.11 2.24"/>
-            </geometry>
-        </collision>
-        <xacro:inertial_box mass="200" x="1.8" y="1.11" z="2.24">
+        </collision>
+        <xacro:inertial_box mass="50" x="1.8" y="1.11" z="2.24">
             <origin xyz="0.9 0 1.12" rpy="0 0 0"/>
         </xacro:inertial_box>
@@ -199,9 +199,10 @@
         <material>Gazebo/Blue</material>
     </gazebo>
+    <!-- 2.3334 -->
     <!-- Cart 2 -->
     <joint name="cart2_joint" type="revolute">
         <parent link="cart"/>
         <child link="cart2"/>
-        <origin xyz="2.3334 0 0" rpy="0 0 0"/>
+        <origin xyz="2.7334 0 0" rpy="0 0 0"/>
         <axis xyz="0 0 1"/>
         <limit effort="10" velocity="1.0" lower="-1.57" upper="1.57"/>
@@ -209,17 +210,17 @@
     <link name="cart2">
         <visual>
+            <origin xyz="0.9 0 0.7" rpy="0 0 0"/>
+            <geometry>
+                <box size="1.8 1.11 1.5"/>
+            </geometry>
+            <material name="white"/>
+        </visual>
+        <collision>
             <origin xyz="0.9 0 1.12" rpy="0 0 0"/>
             <geometry>
                 <box size="1.8 1.11 2.24"/>
             </geometry>
-            <material name="white"/>
-        </visual>
-        <collision>
-            <origin xyz="0.9 0 1.12" rpy="0 0 0"/>
-            <geometry>
-                <box size="1.8 1.11 2.24"/>
-            </geometry>
-        </collision>
-        <xacro:inertial_box mass="200" x="1.8" y="1.11" z="2.24">
+        </collision>
+        <xacro:inertial_box mass="20" x="1.8" y="1.11" z="2.24">
             <origin xyz="0.9 0 1.12" rpy="0 0 0"/>
         </xacro:inertial_box>

Commit message: Modified the carts' collision and inertial geometry to match the visual geometry; physics fixed

File: description/robot_core.xacro (robot description, xacro)
@@ -35,5 +35,5 @@
             </geometry>
         </collision>
-        <xacro:inertial_box mass="100" x="1.645" y="0.8" z="1.8">
+        <xacro:inertial_box mass="50" x="1.645" y="0.8" z="1.8">
             <origin xyz="0.8225 0 0.85" rpy="0 0 0"/>
         </xacro:inertial_box>
@@ -61,5 +61,5 @@
             </geometry>
         </collision>
-        <xacro:inertial_cylinder mass="10" length="0.1" radius="0.2">
+        <xacro:inertial_cylinder mass="5" length="0.1" radius="0.2">
             <origin xyz="0 0 0" rpy="0 0 0"/>
         </xacro:inertial_cylinder>
@@ -87,5 +87,5 @@
             </geometry>
         </collision>
-        <xacro:inertial_cylinder mass="10" length="0.1" radius="0.2">
+        <xacro:inertial_cylinder mass="5" length="0.1" radius="0.2">
             <origin xyz="0 0 0" rpy="0 0 0"/>
         </xacro:inertial_cylinder>
@@ -112,5 +112,5 @@
             </geometry>
         </collision>
-        <xacro:inertial_sphere mass="10" radius="0.1">
+        <xacro:inertial_sphere mass="5" radius="0.1">
             <origin xyz="0 0 0" rpy="0 0 0"/>
         </xacro:inertial_sphere>
@@ -131,7 +131,7 @@
     <link name="cart">
         <visual>
-            <origin xyz="0.9 0 1.12" rpy="0 0 0"/>
-            <geometry>
-                <box size="1.8 1.11 2.24"/>
+            <origin xyz="0.9 0 0.7" rpy="0 0 0"/>
+            <geometry>
+                <box size="1.8 1.11 1.5"/>
             </geometry>
             <material name="white"/>
@@ -140,8 +140,8 @@
             <origin xyz="0.9 0 1.12" rpy="0 0 0"/>
             <geometry>
-                <box size="1.8 1.11 2.24"/>
-            </geometry>
-        </collision>
-        <xacro:inertial_box mass="200" x="1.8" y="1.11" z="2.24">
+                <box size="1.8 1.11 1.5"/>
+            </geometry>
+        </collision>
+        <xacro:inertial_box mass="50" x="1.8" y="1.11" z="1.5">
             <origin xyz="0.9 0 1.12" rpy="0 0 0"/>
         </xacro:inertial_box>
@@ -199,9 +199,10 @@
         <material>Gazebo/Blue</material>
     </gazebo>
+    <!-- 2.3334 -->
     <!-- Cart 2 -->
     <joint name="cart2_joint" type="revolute">
         <parent link="cart"/>
         <child link="cart2"/>
-        <origin xyz="2.3334 0 0" rpy="0 0 0"/>
+        <origin xyz="2.7334 0 0" rpy="0 0 0"/>
         <axis xyz="0 0 1"/>
         <limit effort="10" velocity="1.0" lower="-1.57" upper="1.57"/>
@@ -209,7 +210,7 @@
     <link name="cart2">
         <visual>
-            <origin xyz="0.9 0 1.12" rpy="0 0 0"/>
-            <geometry>
-                <box size="1.8 1.11 2.24"/>
+            <origin xyz="0.9 0 0.7" rpy="0 0 0"/>
+            <geometry>
+                <box size="1.8 1.11 1.5"/>
             </geometry>
             <material name="white"/>
@@ -218,8 +219,8 @@
             <origin xyz="0.9 0 1.12" rpy="0 0 0"/>
             <geometry>
-                <box size="1.8 1.11 2.24"/>
-            </geometry>
-        </collision>
-        <xacro:inertial_box mass="200" x="1.8" y="1.11" z="2.24">
+                <box size="1.8 1.11 1.5"/>
+            </geometry>
+        </collision>
+        <xacro:inertial_box mass="20" x="1.8" y="1.11" z="1.5">
             <origin xyz="0.9 0 1.12" rpy="0 0 0"/>
         </xacro:inertial_box>

Commit message: Modified cart 1 to take the dimensions of bumper doley

File: description/robot_core.xacro (robot description, xacro)
@@ -121,9 +121,9 @@
         <mu2 value="0.15"/>
     </gazebo>
-    <!-- Cart -->
+    <!-- Cart 1: Bumper Doley -->
     <joint name="cart_joint" type="revolute">
         <parent link="chassis"/>
         <child link="cart"/>
-        <origin xyz="-0.5334 0 0" rpy="0 0 ${pi}"/>
+        <origin xyz="-1.5334 0 0" rpy="0 0 ${pi}"/>
         <axis xyz="0 0 1"/>
         <limit effort="10" velocity="1.0" lower="-1.57" upper="1.57"/>
@@ -133,5 +133,5 @@
             <origin xyz="0.9 0 0.7" rpy="0 0 0"/>
             <geometry>
-                <box size="1.8 1.11 1.5"/>
+                <box size="3.315 1.3 1.5"/>
             </geometry>
             <material name="white"/>
@@ -140,8 +140,8 @@
             <origin xyz="0.9 0 1.12" rpy="0 0 0"/>
             <geometry>
-                <box size="1.8 1.11 1.5"/>
-            </geometry>
-        </collision>
-        <xacro:inertial_box mass="50" x="1.8" y="1.11" z="1.5">
+                <box size="3.315 1.3 1.5"/>
+            </geometry>
+        </collision>
+        <xacro:inertial_box mass="50" x="3.315" y="1.3" z="1.5">
             <origin xyz="0.9 0 1.12" rpy="0 0 0"/>
         </xacro:inertial_box>
@@ -151,5 +151,5 @@
         <parent link="cart"/>
         <child link="cart_left_wheel"/>
-        <origin xyz="1.6 0.55 0" rpy="-${pi/2} 0 0"/>
+        <origin xyz="2.2 0.6 0" rpy="-${pi/2} 0 0"/>
         <axis xyz="0 0 1"/>
     </joint>
@@ -177,5 +177,5 @@
         <parent link="cart"/>
         <child link="cart_right_wheel"/>
-        <origin xyz="1.6 -0.55 0" rpy="${pi/2} 0 0"/>
+        <origin xyz="2.2 -0.6 0" rpy="${pi/2} 0 0"/>
         <axis xyz="0 0 -1"/>
     </joint>
@@ -200,5 +200,5 @@
     </gazebo>
     <!-- 2.3334 -->
-    <!-- Cart 2 -->
+    <!-- Cart 2
     <joint name="cart2_joint" type="revolute">
         <parent link="cart"/>
@@ -276,3 +276,4 @@
         <material>Gazebo/Blue</material>
     </gazebo>
+    -->
 </robot>

Commit message: Added cart 2 back to take the dimensions of grill doley

File: description/robot_core.xacro (robot description, xacro)
@@ -200,9 +200,9 @@
     </gazebo>
     <!-- 2.3334 -->
-    <!-- Cart 2
+    <!-- Cart 2 -->
     <joint name="cart2_joint" type="revolute">
         <parent link="cart"/>
         <child link="cart2"/>
-        <origin xyz="2.7334 0 0" rpy="0 0 0"/>
+        <origin xyz="3.2334 0 0" rpy="0 0 0"/>
         <axis xyz="0 0 1"/>
         <limit effort="10" velocity="1.0" lower="-1.57" upper="1.57"/>
@@ -276,4 +276,3 @@
         <material>Gazebo/Blue</material>
     </gazebo>
-    -->
 </robot>

Commit message: Added cart 3 to take the dimensions of s/s doley; Introduced parasitic drifting that must be resolved

File: description/robot_core.xacro (robot description, xacro)
@@ -276,3 +276,79 @@
         <material>Gazebo/Blue</material>
     </gazebo>
+    <!-- Cart 3: S/S Doley -->
+    <joint name="cart3_joint" type="revolute">
+        <parent link="cart2"/>
+        <child link="cart3"/>
+        <origin xyz="2.7334 0 0" rpy="0 0 0"/>
+        <axis xyz="0 0 1"/>
+        <limit effort="10" velocity="1.0" lower="-1.57" upper="1.57"/>
+    </joint>
+    <link name="cart3">
+        <visual>
+            <origin xyz="0.9 0 0.7" rpy="0 0 0"/>
+            <geometry>
+                <box size="2.03 0.765 1.5"/>
+            </geometry>
+            <material name="white"/>
+        </visual>
+        <collision>
+            <origin xyz="0.9 0 1.12" rpy="0 0 0"/>
+            <geometry>
+                <box size="2.03 0.765 1.5"/>
+            </geometry>
+        </collision>
+        <xacro:inertial_box mass="20" x="2.03" y="0.765" z="1.5">
+            <origin xyz="0.9 0 1.12" rpy="0 0 0"/>
+        </xacro:inertial_box>
+    </link>
+    <joint name="cart3_left_wheel_joint" type="continuous">
+        <parent link="cart3"/>
+        <child link="cart3_left_wheel"/>
+        <origin xyz="1.6 0.55 0" rpy="-${pi/2} 0 0"/>
+        <axis xyz="0 0 1"/>
+    </joint>
+    <link name="cart3_left_wheel">
+        <visual>
+            <geometry>
+                <cylinder length="0.2" radius="0.15" />
+            </geometry>
+            <material name="blue"/>
+        </visual>
+        <collision>
+            <geometry>
+                <cylinder length="0.2" radius="0.15" />
+            </geometry>
+        </collision>
+        <xacro:inertial_cylinder mass="5" length="0.2" radius="0.15">
+            <origin xyz="0 0 0" rpy="0 0 0"/>
+        </xacro:inertial_cylinder>
+    </link>
+    <gazebo reference="cart3_left_wheel">
+        <material>Gazebo/Blue</material>
+    </gazebo>
+    <joint name="cart3_right_wheel_joint" type="continuous">
+        <parent link="cart3"/>
+        <child link="cart3_right_wheel"/>
+        <origin xyz="1.6 -0.55 0" rpy="${pi/2} 0 0"/>
+        <axis xyz="0 0 -1"/>
+    </joint>
+    <link name="cart3_right_wheel">
+        <visual>
+            <geometry>
+                <cylinder length="0.2" radius="0.15" />
+            </geometry>
+            <material name="blue"/>
+        </visual>
+        <collision>
+            <geometry>
+                <cylinder length="0.2" radius="0.15" />
+            </geometry>
+        </collision>
+        <xacro:inertial_cylinder mass="5" length="0.2" radius="0.15">
+            <origin xyz="0 0 0" rpy="0 0 0"/>
+        </xacro:inertial_cylinder>
+    </link>
+    <gazebo reference="cart3_right_wheel">
+        <material>Gazebo/Blue</material>
+    </gazebo>
 </robot>

Commit message: Added one cart behind the main robot

File: description/robot_core.xacro (robot description, xacro)
@@ -129,5 +129,5 @@
     </gazebo>
     <!-- CART -->
-    <!-- <joint name="cart_joint" type="revolute">
+    <joint name="cart_joint" type="revolute">
         <parent link="chassis"/>
         <child link="cart"/>
@@ -153,7 +153,7 @@
             <origin xyz="0.15 0 0.075" rpy="0 0 0"/>
         </xacro:inertial_box>
-    </link> -->
+    </link>
     <!-- LEFT WHEEL -->
-    <!-- <joint name="cart_left_wheel_joint" type="continuous">
+    <joint name="cart_left_wheel_joint" type="continuous">
         <parent link="cart"/>
         <child link="cart_left_wheel"/>
@@ -179,7 +179,7 @@
     <gazebo reference="cart_left_wheel">
         <material>Gazebo/Blue</material>
-    </gazebo> -->
+    </gazebo>
     <!-- RIGHT WHEEL -->
-    <!-- <joint name="cart_right_wheel_joint" type="continuous">
+    <joint name="cart_right_wheel_joint" type="continuous">
         <parent link="cart"/>
         <child link="cart_right_wheel"/>
@@ -205,5 +205,5 @@
     <gazebo reference="cart_right_wheel">
         <material>Gazebo/Blue</material>
-    </gazebo> -->
+    </gazebo>
     <!-- CART 2 -->
     <!-- <joint name="cart2_joint" type="revolute">

Commit message: Added second cart to the system

File: description/robot_core.xacro (robot description, xacro)
@@ -207,5 +207,5 @@
     </gazebo>
     <!-- CART 2 -->
-    <!-- <joint name="cart2_joint" type="revolute">
+    <joint name="cart2_joint" type="revolute">
         <parent link="cart"/>
         <child link="cart2"/>
@@ -231,7 +231,7 @@
             <origin xyz="0.15 0 0.075" rpy="0 0 0"/>
         </xacro:inertial_box>
-    </link> -->
+    </link>
     <!-- LEFT WHEEL -->
-    <!-- <joint name="cart2_left_wheel_joint" type="continuous">
+    <joint name="cart2_left_wheel_joint" type="continuous">
         <parent link="cart2"/>
         <child link="cart2_left_wheel"/>
@@ -257,7 +257,7 @@
     <gazebo reference="cart2_left_wheel">
         <material>Gazebo/Blue</material>
-    </gazebo> -->
+    </gazebo>
     <!-- RIGHT WHEEL -->
-    <!-- <joint name="cart2_right_wheel_joint" type="continuous">
+    <joint name="cart2_right_wheel_joint" type="continuous">
         <parent link="cart2"/>
         <child link="cart2_right_wheel"/>
@@ -283,4 +283,4 @@
     <gazebo reference="cart2_right_wheel">
         <material>Gazebo/Blue</material>
-    </gazebo> -->
+    </gazebo>
 </robot>
