Commit message: TEST 2 - Added gazebo_ros_joint_state_publisher to publish robot + cart states. This caused a conflict in joint states between joint_state_broadcaster and gazebo_ros_joint_state_publisher (screenshots attached in multi_cart_system ss folder). Have found three paths to overcome this, trying them next...

File: description/robot_core.xacro (robot description, xacro)
@@ -129,5 +129,5 @@
     </gazebo>
     <!-- CART -->
-    <joint name="cart_joint" type="fixed">
+    <joint name="cart_joint" type="revolute">
         <parent link="chassis"/>
         <child link="cart"/>
@@ -135,4 +135,5 @@
         <axis xyz="0 0 1"/>
         <limit effort="10" velocity="1.0" lower="-1.57" upper="1.57"/>
+        <dynamics damping="0.1" friction="0.0"/>
     </joint>
     <link name="cart">
@@ -154,10 +155,11 @@
         </xacro:inertial_box>
     </link>
-    <!-- LEFT WHEEL -->
-    <joint name="cart_left_wheel_joint" type="fixed">
+    <!-- CART LEFT WHEEL -->
+    <joint name="cart_left_wheel_joint" type="continuous">
         <parent link="cart"/>
         <child link="cart_left_wheel"/>
         <origin xyz="0.28 0.175 0" rpy="-${pi/2} 0 0"/>
         <axis xyz="0 0 1"/>
+        <dynamics damping="0.1" friction="0.0"/>
     </joint>
     <link name="cart_left_wheel">
@@ -177,13 +179,11 @@
         </xacro:inertial_cylinder>
     </link>
-    <gazebo reference="cart_left_wheel">
-        <material>Gazebo/Blue</material>
-    </gazebo>
-    <!-- RIGHT WHEEL -->
-    <joint name="cart_right_wheel_joint" type="fixed">
+    <!-- CART RIGHT WHEEL -->
+    <joint name="cart_right_wheel_joint" type="continuous">
         <parent link="cart"/>
         <child link="cart_right_wheel"/>
         <origin xyz="0.28 -0.175 0" rpy="${pi/2} 0 0"/>
         <axis xyz="0 0 -1"/>
+        <dynamics damping="0.1" friction="0.0"/>
     </joint>
     <link name="cart_right_wheel">
@@ -203,7 +203,88 @@
         </xacro:inertial_cylinder>
     </link>
+    <gazebo reference="cart_left_wheel">
+        <material>Gazebo/Blue</material>
+    </gazebo>
     <gazebo reference="cart_right_wheel">
         <material>Gazebo/Blue</material>
     </gazebo>
+    <!-- CART -->
+    <!-- <joint name="cart_joint" type="fixed">
+        <parent link="chassis"/>
+        <child link="cart"/>
+        <origin xyz="-0.15 0 0" rpy="0 0 ${pi}"/>
+        <axis xyz="0 0 1"/>
+        <limit effort="10" velocity="1.0" lower="-1.57" upper="1.57"/>
+    </joint>
+    <link name="cart">
+        <visual>
+            <origin xyz="0.15 0 0.075" rpy="0 0 0"/>
+            <geometry>
+                <box size="0.3 0.3 0.15"/>
+            </geometry>
+            <material name="white"/>
+        </visual>
+        <collision>
+            <origin xyz="0.15 0 0.075" rpy="0 0 0"/>
+            <geometry>
+                <box size="0.3 0.3 0.15"/>
+            </geometry>
+        </collision>
+        <xacro:inertial_box mass="0.5" x="0.3" y="0.3" z="0.15">
+            <origin xyz="0.15 0 0.075" rpy="0 0 0"/>
+        </xacro:inertial_box>
+    </link> -->
+    <!-- LEFT WHEEL -->
+    <!-- <joint name="cart_left_wheel_joint" type="fixed">
+        <parent link="cart"/>
+        <child link="cart_left_wheel"/>
+        <origin xyz="0.28 0.175 0" rpy="-${pi/2} 0 0"/>
+        <axis xyz="0 0 1"/>
+    </joint>
+    <link name="cart_left_wheel">
+        <visual>
+            <geometry>
+                <cylinder length="0.04" radius="0.05" />
+            </geometry>
+            <material name="blue"/>
+        </visual>
+        <collision>
+            <geometry>
+                <cylinder length="0.04" radius="0.05" />
+            </geometry>
+        </collision>
+        <xacro:inertial_cylinder mass="0.1" length="0.05" radius="0.05">
+            <origin xyz="0 0 0" rpy="0 0 0"/>
+        </xacro:inertial_cylinder>
+    </link>
+    <gazebo reference="cart_left_wheel">
+        <material>Gazebo/Blue</material>
+    </gazebo> -->
+    <!-- RIGHT WHEEL -->
+    <!-- <joint name="cart_right_wheel_joint" type="fixed">
+        <parent link="cart"/>
+        <child link="cart_right_wheel"/>
+        <origin xyz="0.28 -0.175 0" rpy="${pi/2} 0 0"/>
+        <axis xyz="0 0 -1"/>
+    </joint>
+    <link name="cart_right_wheel">
+        <visual>
+            <geometry>
+                <cylinder length="0.04" radius="0.05" />
+            </geometry>
+            <material name="blue"/>
+        </visual>
+        <collision>
+            <geometry>
+                <cylinder length="0.04" radius="0.05" />
+            </geometry>
+        </collision>
+        <xacro:inertial_cylinder mass="0.1" length="0.05" radius="0.05">
+            <origin xyz="0 0 0" rpy="0 0 0"/>
+        </xacro:inertial_cylinder>
+    </link>
+    <gazebo reference="cart_right_wheel">
+        <material>Gazebo/Blue</material>
+    </gazebo> -->
     <!-- CART 2 -->
     <!-- <joint name="cart2_joint" type="revolute">
@@ -284,3 +365,7 @@
         <material>Gazebo/Blue</material>
     </gazebo> -->
+    <!-- gazebo_ros_joint_state_publisher plugin to publish joint states for all joints -->
+    <gazebo>
+        <plugin name="joint_state_publisher" filename="libgazebo_ros_joint_state_publisher.so"/>
+    </gazebo>
 </robot>

Commit message: TEST 3 - SOL_METHOD 1 (FAILED) - Only gazebo_ros_joint_state_publisher, joint_state_broadcaster disabled

File: description/robot_core.xacro (robot description, xacro)
@@ -129,4 +129,85 @@
     </gazebo>
     <!-- CART -->
+    <!-- <joint name="cart_joint" type="revolute">
+        <parent link="chassis"/>
+        <child link="cart"/>
+        <origin xyz="-0.15 0 0" rpy="0 0 ${pi}"/>
+        <axis xyz="0 0 1"/>
+        <limit effort="10" velocity="1.0" lower="-1.57" upper="1.57"/>
+        <dynamics damping="0.1" friction="0.0"/>
+    </joint>
+    <link name="cart">
+        <visual>
+            <origin xyz="0.15 0 0.075" rpy="0 0 0"/>
+            <geometry>
+                <box size="0.3 0.3 0.15"/>
+            </geometry>
+            <material name="white"/>
+        </visual>
+        <collision>
+            <origin xyz="0.15 0 0.075" rpy="0 0 0"/>
+            <geometry>
+                <box size="0.3 0.3 0.15"/>
+            </geometry>
+        </collision>
+        <xacro:inertial_box mass="0.5" x="0.3" y="0.3" z="0.15">
+            <origin xyz="0.15 0 0.075" rpy="0 0 0"/>
+        </xacro:inertial_box>
+    </link> -->
+    <!-- CART LEFT WHEEL -->
+    <!-- <joint name="cart_left_wheel_joint" type="continuous">
+        <parent link="cart"/>
+        <child link="cart_left_wheel"/>
+        <origin xyz="0.28 0.175 0" rpy="-${pi/2} 0 0"/>
+        <axis xyz="0 0 1"/>
+        <dynamics damping="0.1" friction="0.0"/>
+    </joint>
+    <link name="cart_left_wheel">
+        <visual>
+            <geometry>
+                <cylinder length="0.04" radius="0.05" />
+            </geometry>
+            <material name="blue"/>
+        </visual>
+        <collision>
+            <geometry>
+                <cylinder length="0.04" radius="0.05" />
+            </geometry>
+        </collision>
+        <xacro:inertial_cylinder mass="0.1" length="0.05" radius="0.05">
+            <origin xyz="0 0 0" rpy="0 0 0"/>
+        </xacro:inertial_cylinder>
+    </link> -->
+    <!-- CART RIGHT WHEEL -->
+    <!-- <joint name="cart_right_wheel_joint" type="continuous">
+        <parent link="cart"/>
+        <child link="cart_right_wheel"/>
+        <origin xyz="0.28 -0.175 0" rpy="${pi/2} 0 0"/>
+        <axis xyz="0 0 -1"/>
+        <dynamics damping="0.1" friction="0.0"/>
+    </joint>
+    <link name="cart_right_wheel">
+        <visual>
+            <geometry>
+                <cylinder length="0.04" radius="0.05" />
+            </geometry>
+            <material name="blue"/>
+        </visual>
+        <collision>
+            <geometry>
+                <cylinder length="0.04" radius="0.05" />
+            </geometry>
+        </collision>
+        <xacro:inertial_cylinder mass="0.1" length="0.05" radius="0.05">
+            <origin xyz="0 0 0" rpy="0 0 0"/>
+        </xacro:inertial_cylinder>
+    </link>
+    <gazebo reference="cart_left_wheel">
+        <material>Gazebo/Blue</material>
+    </gazebo>
+    <gazebo reference="cart_right_wheel">
+        <material>Gazebo/Blue</material>
+    </gazebo> -->
+    <!-- CART -->
     <joint name="cart_joint" type="revolute">
         <parent link="chassis"/>
@@ -135,5 +216,4 @@
         <axis xyz="0 0 1"/>
         <limit effort="10" velocity="1.0" lower="-1.57" upper="1.57"/>
-        <dynamics damping="0.1" friction="0.0"/>
     </joint>
     <link name="cart">
@@ -155,5 +235,5 @@
         </xacro:inertial_box>
     </link>
-    <!-- CART LEFT WHEEL -->
+    <!-- LEFT WHEEL -->
     <joint name="cart_left_wheel_joint" type="continuous">
         <parent link="cart"/>
@@ -161,5 +241,4 @@
         <origin xyz="0.28 0.175 0" rpy="-${pi/2} 0 0"/>
         <axis xyz="0 0 1"/>
-        <dynamics damping="0.1" friction="0.0"/>
     </joint>
     <link name="cart_left_wheel">
@@ -179,5 +258,8 @@
         </xacro:inertial_cylinder>
     </link>
-    <!-- CART RIGHT WHEEL -->
+    <gazebo reference="cart_left_wheel">
+        <material>Gazebo/Blue</material>
+    </gazebo>
+    <!-- RIGHT WHEEL -->
     <joint name="cart_right_wheel_joint" type="continuous">
         <parent link="cart"/>
@@ -185,5 +267,4 @@
         <origin xyz="0.28 -0.175 0" rpy="${pi/2} 0 0"/>
         <axis xyz="0 0 -1"/>
-        <dynamics damping="0.1" friction="0.0"/>
     </joint>
     <link name="cart_right_wheel">
@@ -203,88 +284,7 @@
         </xacro:inertial_cylinder>
     </link>
-    <gazebo reference="cart_left_wheel">
-        <material>Gazebo/Blue</material>
-    </gazebo>
     <gazebo reference="cart_right_wheel">
         <material>Gazebo/Blue</material>
     </gazebo>
-    <!-- CART -->
-    <!-- <joint name="cart_joint" type="fixed">
-        <parent link="chassis"/>
-        <child link="cart"/>
-        <origin xyz="-0.15 0 0" rpy="0 0 ${pi}"/>
-        <axis xyz="0 0 1"/>
-        <limit effort="10" velocity="1.0" lower="-1.57" upper="1.57"/>
-    </joint>
-    <link name="cart">
-        <visual>
-            <origin xyz="0.15 0 0.075" rpy="0 0 0"/>
-            <geometry>
-                <box size="0.3 0.3 0.15"/>
-            </geometry>
-            <material name="white"/>
-        </visual>
-        <collision>
-            <origin xyz="0.15 0 0.075" rpy="0 0 0"/>
-            <geometry>
-                <box size="0.3 0.3 0.15"/>
-            </geometry>
-        </collision>
-        <xacro:inertial_box mass="0.5" x="0.3" y="0.3" z="0.15">
-            <origin xyz="0.15 0 0.075" rpy="0 0 0"/>
-        </xacro:inertial_box>
-    </link> -->
-    <!-- LEFT WHEEL -->
-    <!-- <joint name="cart_left_wheel_joint" type="fixed">
-        <parent link="cart"/>
-        <child link="cart_left_wheel"/>
-        <origin xyz="0.28 0.175 0" rpy="-${pi/2} 0 0"/>
-        <axis xyz="0 0 1"/>
-    </joint>
-    <link name="cart_left_wheel">
-        <visual>
-            <geometry>
-                <cylinder length="0.04" radius="0.05" />
-            </geometry>
-            <material name="blue"/>
-        </visual>
-        <collision>
-            <geometry>
-                <cylinder length="0.04" radius="0.05" />
-            </geometry>
-        </collision>
-        <xacro:inertial_cylinder mass="0.1" length="0.05" radius="0.05">
-            <origin xyz="0 0 0" rpy="0 0 0"/>
-        </xacro:inertial_cylinder>
-    </link>
-    <gazebo reference="cart_left_wheel">
-        <material>Gazebo/Blue</material>
-    </gazebo> -->
-    <!-- RIGHT WHEEL -->
-    <!-- <joint name="cart_right_wheel_joint" type="fixed">
-        <parent link="cart"/>
-        <child link="cart_right_wheel"/>
-        <origin xyz="0.28 -0.175 0" rpy="${pi/2} 0 0"/>
-        <axis xyz="0 0 -1"/>
-    </joint>
-    <link name="cart_right_wheel">
-        <visual>
-            <geometry>
-                <cylinder length="0.04" radius="0.05" />
-            </geometry>
-            <material name="blue"/>
-        </visual>
-        <collision>
-            <geometry>
-                <cylinder length="0.04" radius="0.05" />
-            </geometry>
-        </collision>
-        <xacro:inertial_cylinder mass="0.1" length="0.05" radius="0.05">
-            <origin xyz="0 0 0" rpy="0 0 0"/>
-        </xacro:inertial_cylinder>
-    </link>
-    <gazebo reference="cart_right_wheel">
-        <material>Gazebo/Blue</material>
-    </gazebo> -->
     <!-- CART 2 -->
     <!-- <joint name="cart2_joint" type="revolute">

Commit message: TEST 4 - SOL_METHOD 2 (failed) - Both publishers online. Only broadcaster works for some reason. Need to explore older code where both of them worked.

File: description/robot_core.xacro (robot description, xacro)
@@ -129,4 +129,85 @@
     </gazebo>
     <!-- CART -->
+    <joint name="cart_joint" type="revolute">
+        <parent link="chassis"/>
+        <child link="cart"/>
+        <origin xyz="-0.15 0 0" rpy="0 0 ${pi}"/>
+        <axis xyz="0 0 1"/>
+        <limit effort="10" velocity="1.0" lower="-1.57" upper="1.57"/>
+        <dynamics damping="0.1" friction="0.0"/>
+    </joint>
+    <link name="cart">
+        <visual>
+            <origin xyz="0.15 0 0.075" rpy="0 0 0"/>
+            <geometry>
+                <box size="0.3 0.3 0.15"/>
+            </geometry>
+            <material name="white"/>
+        </visual>
+        <collision>
+            <origin xyz="0.15 0 0.075" rpy="0 0 0"/>
+            <geometry>
+                <box size="0.3 0.3 0.15"/>
+            </geometry>
+        </collision>
+        <xacro:inertial_box mass="0.5" x="0.3" y="0.3" z="0.15">
+            <origin xyz="0.15 0 0.075" rpy="0 0 0"/>
+        </xacro:inertial_box>
+    </link>
+    <!-- CART LEFT WHEEL -->
+    <joint name="cart_left_wheel_joint" type="continuous">
+        <parent link="cart"/>
+        <child link="cart_left_wheel"/>
+        <origin xyz="0.28 0.175 0" rpy="-${pi/2} 0 0"/>
+        <axis xyz="0 0 1"/>
+        <dynamics damping="0.1" friction="0.0"/>
+    </joint>
+    <link name="cart_left_wheel">
+        <visual>
+            <geometry>
+                <cylinder length="0.04" radius="0.05" />
+            </geometry>
+            <material name="blue"/>
+        </visual>
+        <collision>
+            <geometry>
+                <cylinder length="0.04" radius="0.05" />
+            </geometry>
+        </collision>
+        <xacro:inertial_cylinder mass="0.1" length="0.05" radius="0.05">
+            <origin xyz="0 0 0" rpy="0 0 0"/>
+        </xacro:inertial_cylinder>
+    </link>
+    <!-- CART RIGHT WHEEL -->
+    <joint name="cart_right_wheel_joint" type="continuous">
+        <parent link="cart"/>
+        <child link="cart_right_wheel"/>
+        <origin xyz="0.28 -0.175 0" rpy="${pi/2} 0 0"/>
+        <axis xyz="0 0 -1"/>
+        <dynamics damping="0.1" friction="0.0"/>
+    </joint>
+    <link name="cart_right_wheel">
+        <visual>
+            <geometry>
+                <cylinder length="0.04" radius="0.05" />
+            </geometry>
+            <material name="blue"/>
+        </visual>
+        <collision>
+            <geometry>
+                <cylinder length="0.04" radius="0.05" />
+            </geometry>
+        </collision>
+        <xacro:inertial_cylinder mass="0.1" length="0.05" radius="0.05">
+            <origin xyz="0 0 0" rpy="0 0 0"/>
+        </xacro:inertial_cylinder>
+    </link>
+    <gazebo reference="cart_left_wheel">
+        <material>Gazebo/Blue</material>
+    </gazebo>
+    <gazebo reference="cart_right_wheel">
+        <material>Gazebo/Blue</material>
+    </gazebo>
+    <!-- CART -->
     <!-- <joint name="cart_joint" type="revolute">
         <parent link="chassis"/>
@@ -135,5 +216,4 @@
         <axis xyz="0 0 1"/>
         <limit effort="10" velocity="1.0" lower="-1.57" upper="1.57"/>
-        <dynamics damping="0.1" friction="0.0"/>
     </joint>
     <link name="cart">
@@ -155,5 +235,5 @@
         </xacro:inertial_box>
     </link> -->
-    <!-- CART LEFT WHEEL -->
+    <!-- LEFT WHEEL -->
     <!-- <joint name="cart_left_wheel_joint" type="continuous">
         <parent link="cart"/>
@@ -161,5 +241,4 @@
         <origin xyz="0.28 0.175 0" rpy="-${pi/2} 0 0"/>
         <axis xyz="0 0 1"/>
-        <dynamics damping="0.1" friction="0.0"/>
     </joint>
     <link name="cart_left_wheel">
@@ -178,6 +257,9 @@
             <origin xyz="0 0 0" rpy="0 0 0"/>
         </xacro:inertial_cylinder>
-    </link> -->
-    <!-- CART RIGHT WHEEL -->
+    </link>
+    <gazebo reference="cart_left_wheel">
+        <material>Gazebo/Blue</material>
+    </gazebo> -->
+    <!-- RIGHT WHEEL -->
     <!-- <joint name="cart_right_wheel_joint" type="continuous">
         <parent link="cart"/>
@@ -185,5 +267,4 @@
         <origin xyz="0.28 -0.175 0" rpy="${pi/2} 0 0"/>
         <axis xyz="0 0 -1"/>
-        <dynamics damping="0.1" friction="0.0"/>
     </joint>
     <link name="cart_right_wheel">
@@ -203,88 +284,7 @@
         </xacro:inertial_cylinder>
     </link>
-    <gazebo reference="cart_left_wheel">
-        <material>Gazebo/Blue</material>
-    </gazebo>
     <gazebo reference="cart_right_wheel">
         <material>Gazebo/Blue</material>
     </gazebo> -->
-    <!-- CART -->
-    <joint name="cart_joint" type="revolute">
-        <parent link="chassis"/>
-        <child link="cart"/>
-        <origin xyz="-0.15 0 0" rpy="0 0 ${pi}"/>
-        <axis xyz="0 0 1"/>
-        <limit effort="10" velocity="1.0" lower="-1.57" upper="1.57"/>
-    </joint>
-    <link name="cart">
-        <visual>
-            <origin xyz="0.15 0 0.075" rpy="0 0 0"/>
-            <geometry>
-                <box size="0.3 0.3 0.15"/>
-            </geometry>
-            <material name="white"/>
-        </visual>
-        <collision>
-            <origin xyz="0.15 0 0.075" rpy="0 0 0"/>
-            <geometry>
-                <box size="0.3 0.3 0.15"/>
-            </geometry>
-        </collision>
-        <xacro:inertial_box mass="0.5" x="0.3" y="0.3" z="0.15">
-            <origin xyz="0.15 0 0.075" rpy="0 0 0"/>
-        </xacro:inertial_box>
-    </link>
-    <!-- LEFT WHEEL -->
-    <joint name="cart_left_wheel_joint" type="continuous">
-        <parent link="cart"/>
-        <child link="cart_left_wheel"/>
-        <origin xyz="0.28 0.175 0" rpy="-${pi/2} 0 0"/>
-        <axis xyz="0 0 1"/>
-    </joint>
-    <link name="cart_left_wheel">
-        <visual>
-            <geometry>
-                <cylinder length="0.04" radius="0.05" />
-            </geometry>
-            <material name="blue"/>
-        </visual>
-        <collision>
-            <geometry>
-                <cylinder length="0.04" radius="0.05" />
-            </geometry>
-        </collision>
-        <xacro:inertial_cylinder mass="0.1" length="0.05" radius="0.05">
-            <origin xyz="0 0 0" rpy="0 0 0"/>
-        </xacro:inertial_cylinder>
-    </link>
-    <gazebo reference="cart_left_wheel">
-        <material>Gazebo/Blue</material>
-    </gazebo>
-    <!-- RIGHT WHEEL -->
-    <joint name="cart_right_wheel_joint" type="continuous">
-        <parent link="cart"/>
-        <child link="cart_right_wheel"/>
-        <origin xyz="0.28 -0.175 0" rpy="${pi/2} 0 0"/>
-        <axis xyz="0 0 -1"/>
-    </joint>
-    <link name="cart_right_wheel">
-        <visual>
-            <geometry>
-                <cylinder length="0.04" radius="0.05" />
-            </geometry>
-            <material name="blue"/>
-        </visual>
-        <collision>
-            <geometry>
-                <cylinder length="0.04" radius="0.05" />
-            </geometry>
-        </collision>
-        <xacro:inertial_cylinder mass="0.1" length="0.05" radius="0.05">
-            <origin xyz="0 0 0" rpy="0 0 0"/>
-        </xacro:inertial_cylinder>
-    </link>
-    <gazebo reference="cart_right_wheel">
-        <material>Gazebo/Blue</material>
-    </gazebo>
     <!-- CART 2 -->
     <!-- <joint name="cart2_joint" type="revolute">
