Commit message: Added ultrasonic sensors to right and left directions of cart 1; re-enabled lidar for robot

File: description/robot.urdf.xacro (robot description, xacro)
@@ -3,5 +3,6 @@
     <xacro:include filename="robot_core.xacro" />
     <xacro:include filename="gazebo_control.xacro" />
-    <!--- <xacro:include filename="lidar.xacro" /> -->
-    <xacro:include filename="ultrasonic.xacro" />
+    <xacro:include filename="lidar.xacro" />
+    <xacro:include filename="ultrasonic_t1r1.xacro" />
+    <xacro:include filename="ultrasonic_t1l1.xacro" />
 </robot>

File: description/ultrasonic_t1r1.xacro (robot description, xacro)
@@ -1,31 +1,31 @@
 <?xml version="1.0"?>
 <robot xmlns:xacro="http://www.ros.org/wiki/xacro" >
-    <joint name="ultrasonic_joint" type="fixed">
-        <parent link="chassis"/>
-        <child link="ultrasonic"/>
-        <origin xyz="0.1 0 0.175" rpy="0 0 0"/>
+    <joint name="ultrasonic_t1r1_joint" type="fixed">
+        <parent link="cart"/>
+        <child link="ultrasonic_t1r1"/>
+        <origin xyz="0.15 0.10 0.175" rpy="0 0 ${pi/2}"/>
     </joint>
-    <link name="ultrasonic">
+    <link name="ultrasonic_t1r1">
         <visual>
             <geometry>
-                <cylinder radius="0.01" length="0.02"/>
+                <cylinder radius="0.01" length="0.05"/>
             </geometry>
-            <material name="green"/>
+            <material name="brown"/>
         </visual>
         <collision>
             <geometry>
-                <cylinder radius="0.01" length="0.02"/>
+                <cylinder radius="0.01" length="0.05"/>
             </geometry>
         </collision>
-        <xacro:inertial_cylinder mass="0.1" length="0.02" radius="0.01">
+        <xacro:inertial_cylinder mass="0.1" length="0.05" radius="0.01">
             <origin xyz="0 0 0" rpy="0 0 0"/>
         </xacro:inertial_cylinder>
     </link>
-    <material name="green">
+    <material name="brown">
         <color rgba="1 0 0 1"/>
     </material>
-    <gazebo reference="ultrasonic">
-        <material>Gazebo/Green</material>
-        <sensor name="ultrasonic" type="ray">
+    <gazebo reference="ultrasonic_t1r1">
+        <material>Gazebo/Brown</material>
+        <sensor name="ultrasonic_t1r1" type="ray">
             <pose> 0 0 0 0 0 0 </pose>
             <visualize>true</visualize>
@@ -44,10 +44,10 @@
                 </range>
             </ray>
-            <plugin name="ultrasonic_controller" filename="libgazebo_ros_ray_sensor.so">
+            <plugin name="ultrasonic_t1r1_controller" filename="libgazebo_ros_ray_sensor.so">
                 <ros>
                     <argument>~/out:=scan</argument>
                 </ros>
                 <output_type>sensor_msgs/LaserScan</output_type>
-                <frame_name>ultrasonic</frame_name>
+                <frame_name>ultrasonic_t1r1</frame_name>
             </plugin>
         </sensor>

Commit message: Trial 1

File: description/robot.urdf.xacro (robot description, xacro)
@@ -3,6 +3,6 @@
     <xacro:include filename="robot_core.xacro" />
     <xacro:include filename="gazebo_control.xacro" />
-    <xacro:include filename="lidar.xacro" />
-    <xacro:include filename="ultrasonic_t1r1.xacro" />
-    <xacro:include filename="ultrasonic_t1l1.xacro" />
+    <!-- <xacro:include filename="lidar.xacro" /> -->
+    <!-- <xacro:include filename="ultrasonic_t1r1.xacro" /> -->
+    <!-- <xacro:include filename="ultrasonic_t1l1.xacro" /> -->
 </robot>

File: description/robot_core.xacro (robot description, xacro)
@@ -19,22 +19,22 @@
         <parent link="base_link"/>
         <child link="chassis"/>
-        <origin xyz="-0.1 0 0"/>
+        <origin xyz="-0.3 0 0"/>
     </joint>
     <link name="chassis">
         <visual>
-            <origin xyz="0.15 0 0.075" rpy="0 0 0"/>
-            <geometry>
-                <box size="0.3 0.3 0.15"/>
+            <origin xyz="0.8225 0 1.0" rpy="0 0 0"/>
+            <geometry>
+                <box size="1.645 0.8 2"/>
             </geometry>
             <material name="white"/>
         </visual>
         <collision>
-            <origin xyz="0.15 0 0.075" rpy="0 0 0"/>
-            <geometry>
-                <box size="0.3 0.3 0.15"/>
-            </geometry>
-        </collision>
-        <xacro:inertial_box mass="0.5" x="0.3" y="0.3" z="0.15">
-            <origin xyz="0.15 0 0.075" rpy="0 0 0"/>
+            <origin xyz="0.8225 0 1.0" rpy="0 0 0"/>
+            <geometry>
+                <box size="1.645 0.8 2"/>
+            </geometry>
+        </collision>
+        <xacro:inertial_box mass="50" x="1.645" y="0.8" z="2">
+            <origin xyz="0.8225 0 1.0" rpy="0 0 0"/>
         </xacro:inertial_box>
     </link>
@@ -46,5 +46,5 @@
         <parent link="base_link"/>
         <child link="left_wheel"/>
-        <origin xyz="0 0.175 0" rpy="-${pi/2} 0 0"/>
+        <origin xyz="0 0.4 0.2" rpy="-${pi/2} 0 0"/>
         <axis xyz="0 0 1"/>
     </joint>
@@ -52,14 +52,14 @@
         <visual>
             <geometry>
-                <cylinder length="0.04" radius="0.05" />
-            </geometry>
-            <material name="blue"/>
-        </visual>
-        <collision>
-            <geometry>
-                <cylinder length="0.04" radius="0.05" />
-            </geometry>
-        </collision>
-        <xacro:inertial_cylinder mass="0.1" length="0.05" radius="0.05">
+                <cylinder length="0.1" radius="0.2" />
+            </geometry>
+            <material name="blue"/>
+        </visual>
+        <collision>
+            <geometry>
+                <cylinder length="0.1" radius="0.2" />
+            </geometry>
+        </collision>
+        <xacro:inertial_cylinder mass="5" length="0.1" radius="0.2">
             <origin xyz="0 0 0" rpy="0 0 0"/>
         </xacro:inertial_cylinder>
@@ -72,5 +72,5 @@
         <parent link="base_link"/>
         <child link="right_wheel"/>
-        <origin xyz="0 -0.175 0" rpy="${pi/2} 0 0"/>
+        <origin xyz="0 -0.4 0.2" rpy="${pi/2} 0 0"/>
         <axis xyz="0 0 -1"/>
     </joint>
@@ -78,14 +78,14 @@
         <visual>
             <geometry>
-                <cylinder length="0.04" radius="0.05" />
-            </geometry>
-            <material name="blue"/>
-        </visual>
-        <collision>
-            <geometry>
-                <cylinder length="0.04" radius="0.05" />
-            </geometry>
-        </collision>
-        <xacro:inertial_cylinder mass="0.1" length="0.05" radius="0.05">
+                <cylinder length="0.1" radius="0.2" />
+            </geometry>
+            <material name="blue"/>
+        </visual>
+        <collision>
+            <geometry>
+                <cylinder length="0.1" radius="0.2" />
+            </geometry>
+        </collision>
+        <xacro:inertial_cylinder mass="5" length="0.1" radius="0.2">
             <origin xyz="0 0 0" rpy="0 0 0"/>
         </xacro:inertial_cylinder>
@@ -98,10 +98,10 @@
         <parent link="chassis"/>
         <child link="caster_wheel"/>
-        <origin xyz="0.24 0 -0.03" rpy="0 0 0"/>
+        <origin xyz="1.2 0 -0.1" rpy="0 0 0"/>
     </joint>
     <link name="caster_wheel">
         <visual>
             <geometry>
-                <sphere radius="0.05" />
+                <sphere radius="0.1" />
             </geometry>
             <material name="black"/>
@@ -109,8 +109,8 @@
         <collision>
             <geometry>
-                <cylinder length="0.04" radius="0.05" />
-            </geometry>
-        </collision>
-        <xacro:inertial_sphere mass="0.1" radius="0.05">
+                <sphere radius="0.1" />
+            </geometry>
+        </collision>
+        <xacro:inertial_sphere mass="2" radius="0.1">
             <origin xyz="0 0 0" rpy="0 0 0"/>
         </xacro:inertial_sphere>
@@ -121,5 +121,5 @@
         <mu2 value="0.5"/>
     </gazebo>
-    <!-- CART -->
+    <!--
     <joint name="cart_joint" type="revolute">
         <parent link="chassis"/>
@@ -147,5 +147,4 @@
         </xacro:inertial_box>
     </link>
-    <!-- LEFT WHEEL -->
     <joint name="cart_left_wheel_joint" type="continuous">
         <parent link="cart"/>
@@ -173,5 +172,4 @@
         <material>Gazebo/Blue</material>
     </gazebo>
-    <!-- RIGHT WHEEL -->
     <joint name="cart_right_wheel_joint" type="continuous">
         <parent link="cart"/>
@@ -199,5 +197,4 @@
         <material>Gazebo/Blue</material>
     </gazebo>
-<!-- CART 2 -->
     <joint name="cart2_joint" type="revolute">
         <parent link="cart"/>
@@ -225,5 +222,4 @@
         </xacro:inertial_box>
     </link>
-    <!-- LEFT WHEEL -->
     <joint name="cart2_left_wheel_joint" type="continuous">
         <parent link="cart2"/>
@@ -251,5 +247,4 @@
         <material>Gazebo/Blue</material>
     </gazebo>
-    <!-- RIGHT WHEEL -->
     <joint name="cart2_right_wheel_joint" type="continuous">
         <parent link="cart2"/>
@@ -277,3 +272,4 @@
         <material>Gazebo/Blue</material>
     </gazebo>
+    -->
 </robot>

Commit message: SLAM works perfectly now after removing trailers and ultrasonic sensors. Screenshots added in Run 5.

File: description/robot.urdf.xacro (robot description, xacro)
@@ -5,5 +5,5 @@
     <xacro:include filename="ros2_control.xacro" />
     <xacro:include filename="lidar.xacro" />
-    <xacro:include filename="ultrasonic_t1r1.xacro" />
-    <xacro:include filename="ultrasonic_t1l1.xacro" />
+    <!-- <xacro:include filename="ultrasonic_t1r1.xacro" />
+    <xacro:include filename="ultrasonic_t1l1.xacro" /> -->
 </robot>

File: description/robot_core.xacro (robot description, xacro)
@@ -129,5 +129,5 @@
     </gazebo>
     <!-- CART -->
-    <joint name="cart_joint" type="revolute">
+    <!-- <joint name="cart_joint" type="revolute">
         <parent link="chassis"/>
         <child link="cart"/>
@@ -153,7 +153,7 @@
             <origin xyz="0.15 0 0.075" rpy="0 0 0"/>
         </xacro:inertial_box>
-    </link>
+    </link> -->
     <!-- LEFT WHEEL -->
-    <joint name="cart_left_wheel_joint" type="continuous">
+    <!-- <joint name="cart_left_wheel_joint" type="continuous">
         <parent link="cart"/>
         <child link="cart_left_wheel"/>
@@ -179,7 +179,7 @@
     <gazebo reference="cart_left_wheel">
         <material>Gazebo/Blue</material>
-    </gazebo>
+    </gazebo> -->
     <!-- RIGHT WHEEL -->
-    <joint name="cart_right_wheel_joint" type="continuous">
+    <!-- <joint name="cart_right_wheel_joint" type="continuous">
         <parent link="cart"/>
         <child link="cart_right_wheel"/>
@@ -205,7 +205,7 @@
     <gazebo reference="cart_right_wheel">
         <material>Gazebo/Blue</material>
-    </gazebo>
-<!-- CART 2 -->
-    <joint name="cart2_joint" type="revolute">
+    </gazebo> -->
+    <!-- CART 2 -->
+    <!-- <joint name="cart2_joint" type="revolute">
         <parent link="cart"/>
         <child link="cart2"/>
@@ -231,7 +231,7 @@
             <origin xyz="0.15 0 0.075" rpy="0 0 0"/>
         </xacro:inertial_box>
-    </link>
+    </link> -->
     <!-- LEFT WHEEL -->
-    <joint name="cart2_left_wheel_joint" type="continuous">
+    <!-- <joint name="cart2_left_wheel_joint" type="continuous">
         <parent link="cart2"/>
         <child link="cart2_left_wheel"/>
@@ -257,7 +257,7 @@
     <gazebo reference="cart2_left_wheel">
         <material>Gazebo/Blue</material>
-    </gazebo>
+    </gazebo> -->
     <!-- RIGHT WHEEL -->
-    <joint name="cart2_right_wheel_joint" type="continuous">
+    <!-- <joint name="cart2_right_wheel_joint" type="continuous">
         <parent link="cart2"/>
         <child link="cart2_right_wheel"/>
@@ -283,4 +283,4 @@
     <gazebo reference="cart2_right_wheel">
         <material>Gazebo/Blue</material>
-    </gazebo>
+    </gazebo> -->
 </robot>

Commit message: TEST 1 - Changed cart joint type from "revolute" to "fixed" and wheel joints' type from "continuous" to "fixed" as well. TF issues seem to be resolved. Enabling ultrasonic sensors seems to work roughly as expected as well (some tuning needed there). Of course, fixed joints are not representative of the actual system so need to come up with a more elegant solution.

File: description/robot.urdf.xacro (robot description, xacro)
@@ -5,5 +5,5 @@
     <xacro:include filename="ros2_control.xacro" />
     <xacro:include filename="lidar.xacro" />
-    <!-- <xacro:include filename="ultrasonic_t1r1.xacro" />
-    <xacro:include filename="ultrasonic_t1l1.xacro" /> -->
+    <xacro:include filename="ultrasonic_t1r1.xacro" />
+    <xacro:include filename="ultrasonic_t1l1.xacro" />
 </robot>

File: description/robot_core.xacro (robot description, xacro)
@@ -129,5 +129,5 @@
     </gazebo>
     <!-- CART -->
-    <joint name="cart_joint" type="revolute">
+    <joint name="cart_joint" type="fixed">
         <parent link="chassis"/>
         <child link="cart"/>
@@ -155,5 +155,5 @@
     </link>
     <!-- LEFT WHEEL -->
-    <joint name="cart_left_wheel_joint" type="continuous">
+    <joint name="cart_left_wheel_joint" type="fixed">
         <parent link="cart"/>
         <child link="cart_left_wheel"/>
@@ -181,5 +181,5 @@
     </gazebo>
     <!-- RIGHT WHEEL -->
-    <joint name="cart_right_wheel_joint" type="continuous">
+    <joint name="cart_right_wheel_joint" type="fixed">
         <parent link="cart"/>
         <child link="cart_right_wheel"/>

Commit message: Removed ros2_control, joint_state_broadcaster, and diff_drive_controller to implement gazebo_ros_joint_state_publisher to publish all dynamic joint states. The new publisher is giving plugin missing errors - resolution in progress

File: description/robot.urdf.xacro (robot description, xacro)
@@ -3,7 +3,7 @@
     <xacro:include filename="robot_core.xacro" />
     <!-- <xacro:include filename="gazebo_control.xacro" /> -->
-    <xacro:include filename="ros2_control.xacro" />
-    <xacro:include filename="lidar.xacro" />
+    <!-- <xacro:include filename="ros2_control.xacro" /> -->
+    <!-- <xacro:include filename="lidar.xacro" />
     <xacro:include filename="ultrasonic_t1r1.xacro" />
-    <xacro:include filename="ultrasonic_t1l1.xacro" />
+    <xacro:include filename="ultrasonic_t1l1.xacro" /> -->
 </robot>

File: description/robot_core.xacro (robot description, xacro)
@@ -129,5 +129,5 @@
     </gazebo>
     <!-- CART -->
-    <joint name="cart_joint" type="fixed">
+    <joint name="cart_joint" type="revolute">
         <parent link="chassis"/>
         <child link="cart"/>
@@ -155,5 +155,5 @@
     </link>
     <!-- LEFT WHEEL -->
-    <joint name="cart_left_wheel_joint" type="fixed">
+    <joint name="cart_left_wheel_joint" type="continuous">
         <parent link="cart"/>
         <child link="cart_left_wheel"/>
@@ -181,5 +181,5 @@
     </gazebo>
     <!-- RIGHT WHEEL -->
-    <joint name="cart_right_wheel_joint" type="fixed">
+    <joint name="cart_right_wheel_joint" type="continuous">
         <parent link="cart"/>
         <child link="cart_right_wheel"/>
@@ -284,3 +284,9 @@
         <material>Gazebo/Blue</material>
     </gazebo> -->
+    <!-- gazebo_ros_joint_state_publisher plugin to publish joint states for all joints -->
+    <gazebo>
+        <plugin name="joint_state_publisher" filename="libgazebo_ros_joint_state_publisher.so">
+            <joint_names>left_wheel_joint right_wheel_joint cart_joint cart_left_wheel_joint cart_right_wheel_joint</joint_names>
+        </plugin>
+    </gazebo>
 </robot>

File: description/ros2_control.xacro (robot description, xacro)
@@ -1,5 +1,5 @@
 <?xml version="1.0"?>
 <robot xmlns:xacro="http://www.ros.org/wiki/xacro">
-    <ros2_control name="GazeboSystem" type="system">
+    <!-- <ros2_control name="GazeboSystem" type="system">
     <hardware>
         <plugin>gazebo_ros2_control/GazeboSystem</plugin>
@@ -15,9 +15,9 @@
         <state_interface name="position"/>
     </joint>
-    </ros2_control>
-    <gazebo>
+    </ros2_control> -->
+    <!-- <gazebo>
     <plugin name="gazebo_ros2_control" filename="libgazebo_ros2_control.so">
         <parameters>$(find diff_drive_robot)/config/my_controllers.yaml</parameters>
     </plugin>
-    </gazebo>
+    </gazebo> -->
 </robot>
